File: Kc/MakerLAB_r03/Gen_Clock.kicad_sch (KiCad schematic)
At the start: 17 parts, among them J17 Conn_02x10_Counter_Clockwise, J26 Conn_01x06_Female, SW5 SW_Rotary12, U7 NE555P

Commit message: 20230309-Update
Lavoro in tandem con Marco
Parts:
- *C16: value (none) -> 330pF; footprint (none) -> Capacitor_THT:C_Axial_L5.1mm_D3.1mm_P7.50mm_Horizontal
- J26: footprint (none) -> Connector_PinHeader_2.54mm:PinHeader_1x06_P2.54mm_Vertical
- RV3: footprint (none) -> Potentiometer_THT:Potentiometer_Bourns_3266W_Vertical
- U7: footprint (none) -> Package_DIP:DIP-8_W7.62mm
Changed lines of the file:
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@@
     (property "Reference" "J26" (id 0) (at 97.79 138.43 90))
     (property "Value" "Conn_01x06_Female" (id 1) (at 97.79 140.97 90))
-    (property "Footprint" "" (id 2) (at 99.06 135.89 0)
+    (property "Footprint" "Connector_PinHeader_2.54mm:PinHeader_1x06_P2.54mm_Vertical" (id 2) (at 99.06 135.89 0)
       (effects (font (size 1.27 1.27)) hide)
     )
@@
       (effects (font (size 1.27 1.27)) (justify left))
     )
-    (property "Value" "" (id 1) (at 100.33 153.67 0)
-      (effects (font (size 1.27 1.27)) (justify left))
-    )
-    (property "Footprint" "" (id 2) (at 101.6 152.7048 0)
+    (property "Value" "330pF" (id 1) (at 100.33 153.67 0)
+      (effects (font (size 1.27 1.27)) (justify left))
+    )
+    (property "Footprint" "Capacitor_THT:C_Axial_L5.1mm_D3.1mm_P7.50mm_Horizontal" (id 2) (at 101.6 152.7048 0)
       (effects (font (size 1.27 1.27)) hide)
     )
@@
       (effects (font (size 1.27 1.27)) (justify left))
     )
-    (property "Footprint" "" (id 2) (at 127 71.12 0)
+    (property "Footprint" "Package_DIP:DIP-8_W7.62mm" (id 2) (at 127 71.12 0)
       (effects (font (size 1.27 1.27)) hide)
     )
@@
       (effects (font (size 1.27 1.27)) (justify right))
     )
-    (property "Footprint" "" (id 2) (at 64.77 74.93 0)
-      (effects (font (size 1.27 1.27)) hide)
-    )
+    (property "Footprint" "Potentiometer_THT:Potentiometer_Bourns_3266W_Vertical" (id 2) (at 64.77 74.93 0)
+      (effects (font (size 1.27 1.27)) hide)
+    )
