File: Kc/MakerLAB_r03/Input_8bit.kicad_sch (KiCad schematic)
At the start: 4 parts, among them J15 Conn_01x10_Female, SW2 SW_DIP_x08

Commit message: 20230309-Update
Lavoro in tandem con Marco
Parts:
- C10: footprint (none) -> Capacitor_THT:C_Disc_D7.0mm_W2.5mm_P5.00mm
- J15: value Conn_01x10_Female -> GND 0 1 2 3 4 5 6 7 +5V; footprint (none) -> Connector_PinSocket_2.54mm:PinSocket_1x10_P2.54mm_Vertical
Connections:
- net GND renamed GNDPWR
Other:
- moved on the sheet: C10, J15, RN2, SW2
