File: Kc/MakerLAB_r03/MPU_socket.kicad_sch (KiCad schematic)
At the start: 5 parts, among them J21 Conn_02x20_Counter_Clockwise, J22 Conn_02x20_Counter_Clockwise, J23 Conn_02x20_Counter_Clockwise, J24 Conn_02x20_Counter_Clockwise, J25 Conn_02x20_Counter_Clockwise

Commit message: 20230309-Update
Lavoro in tandem con Marco
Parts:
- removed J21, J25: Conn_02x20_Counter_Clockwise, Connector_PinSocket_2.54mm:PinSocket_2x20_P2.54mm_Vertical, symbol Connector_Generic:Conn_02x20_Odd_Even
