File: Kc/MakerLAB_r03/Tastiera4x4.kicad_sch (KiCad schematic)
At the start: 1 part

Commit message: 20230309-Update
Lavoro in tandem con Marco
Parts:
- J27: renamed from J?; value (none) -> Conn_01x10_Male
Changed lines of the file:
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@@
   (symbol (lib_id "power:GND") (at 40.005 84.455 0) (unit 1)
     (in_bom yes) (on_board yes) (fields_autoplaced)
-    (property "Reference" "#PWR?" (id 0) (at 40.005 90.805 0)
+    (property "Reference" "#PWR0103" (id 0) (at 40.005 90.805 0)
       (effects (font (size 1.27 1.27)) hide)
     )
-    (property "Value" "" (id 1) (at 40.005 88.9 0))
+    (property "Value" "GND" (id 1) (at 40.005 88.9 0))
     (property "Footprint" "" (id 2) (at 40.005 84.455 0)
       (effects (font (size 1.27 1.27)) hide)
@@
   (symbol (lib_id "Connector:Conn_01x10_Male") (at 34.925 70.485 0) (mirror x) (unit 1)
     (in_bom yes) (on_board yes) (fields_autoplaced)
-    (property "Reference" "J?" (id 0) (at 33.02 67.9449 0)
+    (property "Reference" "J27" (id 0) (at 33.02 67.9449 0)
       (effects (font (size 1.27 1.27)) (justify right))
     )
-    (property "Value" "" (id 1) (at 33.02 70.4849 0)
+    (property "Value" "Conn_01x10_Male" (id 1) (at 33.02 70.4849 0)
       (effects (font (size 1.27 1.27)) (justify right))
     )
@@
   (symbol (lib_id "power:+5V") (at 40.005 52.07 0) (unit 1)
     (in_bom yes) (on_board yes) (fields_autoplaced)
-    (property "Reference" "#PWR?" (id 0) (at 40.005 55.88 0)
+    (property "Reference" "#PWR0104" (id 0) (at 40.005 55.88 0)
       (effects (font (size 1.27 1.27)) hide)
     )
-    (property "Value" "" (id 1) (at 40.005 46.99 0))
+    (property "Value" "+5V" (id 1) (at 40.005 46.99 0))
     (property "Footprint" "" (id 2) (at 40.005 52.07 0)
       (effects (font (size 1.27 1.27)) hide)
