File: Kc/MakerLAB_r03/Visual_4Dgt.kicad_sch (KiCad schematic)
At the start: 21 parts, among them J10 Conn_01x02_Female, J11 Conn_02x10_Counter_Clockwise, J12 Conn_02x05_Counter_Clockwise, J9 Conn_02x05_Counter_Clockwise, Q1 2N3904, Q2 2N3904, Q3 2N3904, Q4 2N3904, U3 DM9368, U4 CC56-12EWA

Commit message: 20230309-Update
Lavoro in tandem con Marco
Changed lines of the file:
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@@
       (effects (font (size 1.27 1.27)) hide)
     )
-    (property "Value" "" (id 1) (at 178.435 97.79 0))
+    (property "Value" "GND" (id 1) (at 178.435 97.79 0))
     (property "Footprint" "" (id 2) (at 178.435 92.71 0)
       (effects (font (size 1.27 1.27)) hide)
