File: Kc/MakerLAB_r03/Visual_8Led.kicad_sch (KiCad schematic)
At the start: 21 parts, among them J13 Conn_01x10_Female, J14 Conn_02x10_Counter_Clockwise, U5 ULN2803A

Commit message: 20230309-Update
Lavoro in tandem con Marco
Parts:
- D10: value LED -> 4
- D11: value LED -> 3
- D12: value LED -> 2
- D13: value LED -> 1
- D14: value LED -> 0
- D7: value LED -> 7
- D8: value LED -> 6
- D9: value LED -> 5
- J13: value Conn_01x10_Female -> GND 0 1 2 3 4 5 6 7 +5V
- J14: value Conn_02x10_Counter_Clockwise -> 8Bit Jumper
- RN1: value R_Pack08 -> Resistor Array
- TP10: value TestPoint -> Bit4
- TP11: value TestPoint -> Bit5
- TP12: value TestPoint -> Bit6
- TP13: value TestPoint -> Bit7
- TP6: value TestPoint -> Bit0
- TP7: value TestPoint -> Bit1
- TP8: value TestPoint -> Bit2
- TP9: value TestPoint -> Bit3
Other:
- moved on the sheet: C9, D10, D11, D12, D13, D14, D7, D8, D9, J13, J14, RN1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
