File: Kc/MakerLAB_r03/MakerLAB_r03.kicad_pcb (KiCad board)
At the start: 2 copper layers, 374 x 178 mm, 87 parts, among them J10 Conn_01x02_Female, J11 Conn_02x10_Counter_Clockwise, J12 Conn_02x05_Counter_Clockwise, J13 Conn_01x10_Female, J14 Conn_02x10_Counter_Clockwise, J16 Conn_02x05_Counter_Clockwise, J18 Conn_02x05_Counter_Clockwise, J19 Conn_01x10_Female, J20 Screw_Terminal_01x02, J21 Conn_02x20_Counter_Clockwise, J22 Conn_02x20_Counter_Clockwise, J23 Conn_02x20_Counter_Clockwise, J24 Conn_02x20_Counter_Clockwise, J25 Conn_02x20_Counter_Clockwise, J4 Barrel_Jack_MountingPin, J5 Conn_01x03, J6 Conn_01x03, J7 Conn_01x03, J8 Conn_01x03, J9 Conn_02x05_Counter_Clockwise, Q1 2N3904, Q2 2N3904, Q3 2N3904, Q4 2N3904, SW1 SwGenerale, SW2 SW_DIP_x08, U1 LM317_TO-220, U10 9368, U2 LM7805_TO220, U3 DM9368, U4 CC56-12EWA, U5 ULN2803A, U7 NE555P, U9 9368

Commit message: 20230309-Update
Lavoro in tandem con Marco
Parts:
- removed J21, J25: Conn_02x20_Counter_Clockwise, Connector_PinSocket_2.54mm:PinSocket_2x20_P2.54mm_Vertical
- added C10: 100nF, Capacitor_THT:C_Disc_D7.0mm_W2.5mm_P5.00mm, F.Cu at (139.7, 222.0)
- added C16: 100nF, Capacitor_THT:C_Disc_D7.0mm_W2.5mm_P5.00mm, F.Cu at (-126.7, 65.2)
- added C23: 100nF, Capacitor_THT:C_Disc_D7.0mm_W2.5mm_P5.00mm, F.Cu at (-146.7, 84.8)
- added C24: 100nF, Capacitor_THT:C_Disc_D7.0mm_W2.5mm_P5.00mm, F.Cu at (-158.1, 89.4)
- added C25: 220uF, Capacitor_THT:CP_Radial_D10.0mm_P5.00mm, F.Cu at (-158.6, 71.9)
- added C3: 100nF, Capacitor_THT:C_Disc_D7.0mm_W2.5mm_P5.00mm, F.Cu at (-146.7, 76.7)
- added C4: 10uF, Capacitor_THT:CP_Radial_D5.0mm_P2.00mm, F.Cu at (-139.3, 90.1)
- added C7: 220uF, Capacitor_THT:CP_Radial_D10.0mm_P5.00mm, F.Cu at (-141.4, 59.2)
- added J15: GND 0 1 2 3 4 5 6 7 +5V, Connector_PinSocket_2.54mm:PinSocket_1x10_P2.54mm_Vertical, F.Cu at (119.4, 94.4)
- added J26: Conn_01x06_Female, Connector_PinHeader_2.54mm:PinHeader_1x06_P2.54mm_Vertical, F.Cu at (160.8, 88.9)
- added J28: Conn_01x03, Connector_PinHeader_2.54mm:PinHeader_1x03_P2.54mm_Vertical, F.Cu at (-130.8, 55.8)
- added J29: Conn_01x02_Male, Connector_PinSocket_2.54mm:PinSocket_1x02_P2.54mm_Vertical, F.Cu at (-133.5, 75.2)
- added J30: Conn_01x02_Male, Connector_PinSocket_2.54mm:PinSocket_1x02_P2.54mm_Vertical, F.Cu at (-116.9, 55.8)
- added J31: Conn_01x03, Connector_PinHeader_2.54mm:PinHeader_1x03_P2.54mm_Vertical, F.Cu at (-150.8, 80.0)
- added J32: Conn_01x03, Connector_PinHeader_2.54mm:PinHeader_1x03_P2.54mm_Vertical, F.Cu at (-130.8, 65.5)
- added Q5: 2N3904, Package_TO_SOT_THT:TO-92_Inline, F.Cu at (-119.6, 73.3)
- added RV3: 220K, Potentiometer_THT:Potentiometer_Bourns_3266W_Vertical, F.Cu at (169.8, 88.4)
- added TP14: VarA+, TestPoint:TestPoint_Loop_D3.80mm_Drill2.8mm, F.Cu at (-145.1, 90.3)
- added TP15: VarA-, TestPoint:TestPoint_Loop_D3.80mm_Drill2.8mm, F.Cu at (-136.5, 83.4)
- added TP16: 5VA+, TestPoint:TestPoint_Loop_D3.80mm_Drill2.8mm, F.Cu at (-127.8, 77.5)
- added TP17: 3.3VA+, TestPoint:TestPoint_Loop_D3.80mm_Drill2.8mm, F.Cu at (-106.6, 56.9)
- added TP18: 5VA-, TestPoint:TestPoint_Loop_D3.80mm_Drill2.8mm, F.Cu at (-125.0, 70.6)
- added TP19: 3.3VA-, TestPoint:TestPoint_Loop_D3.80mm_Drill2.8mm, F.Cu at (-116.5, 66.6)
- added U11: L78L33_SOT89, Package_TO_SOT_SMD:SOT-223, F.Cu at (-145.4, 70.2)
- added Uni-A4: Jumper_3_Open, Connector_PinSocket_2.54mm:PinSocket_1x03_P2.54mm_Vertical, F.Cu at (182.1, 88.9)
- C1: footprint Capacitor_THT:CP_Axial_L37.0mm_D13.0mm_P43.00mm_Horizontal -> Capacitor_THT:CP_Radial_D17.0mm_P7.50mm
- C2, C5: footprint Capacitor_THT:C_Axial_L5.1mm_D3.1mm_P7.50mm_Horizontal -> Capacitor_THT:C_Disc_D7.0mm_W2.5mm_P5.00mm
- C6: value 10uF -> 220uF; footprint Capacitor_THT:CP_Axial_L37.0mm_D13.0mm_P43.00mm_Horizontal -> Capacitor_THT:CP_Radial_D10.0mm_P5.00mm
- D10: value LED -> 4
- D11: value LED -> 3
- D12: value LED -> 2
- D13: value LED -> 1
- D14: value LED -> 0
- D7: value LED -> 7
- D8: value LED -> 6
- D9: value LED -> 5
- J13: value Conn_01x10_Female -> GND 0 1 2 3 4 5 6 7 +5V
- J14: value Conn_02x10_Counter_Clockwise -> 8Bit Jumper
- J5: value Conn_01x03 -> Conn_01x02_Male; footprint Connector_PinHeader_2.54mm:PinHeader_1x03_P2.54mm_Vertical -> Connector_PinSocket_2.54mm:PinSocket_1x02_P2.54mm_Vertical
- RN1: value R_Pack08 -> Resistor Array
- TP10: value TestPoint -> Bit4
- TP11: value TestPoint -> Bit5
- TP12: value TestPoint -> Bit6
- TP13: value TestPoint -> Bit7
- TP6: value TestPoint -> Bit0
- TP7: value TestPoint -> Bit1
- TP8: value TestPoint -> Bit2
- TP9: value TestPoint -> Bit3
- moved R3 192.9 mm to (-71.8, 171.3), turned to 0 degrees
- moved H1 180.7 mm to (-34.8, 173.0)
- moved J10 180.7 mm to (-37.2, 166.0)
- moved C8 180.7 mm to (-80.7, 150.2)
- moved D6 180.7 mm to (-46.6, 158.2)
- moved H2 180.7 mm to (-30.8, 186.3)
- moved H3 180.7 mm to (-38.9, 159.7)
- moved *C16 84.1 mm to (126.1, 160.8)
- moved C20 84.1 mm to (136.8, 160.8)
- moved C17 84.1 mm to (126.1, 165.5)
- moved C19 84.1 mm to (126.1, 170.1)
- moved C18 84.1 mm to (136.8, 165.5)
- moved SW2 74.6 mm to (116.8, 51.3), turned to -90 degrees
- moved C22 66.0 mm to (-98.1, 64.2)
- moved RN2 66.0 mm to (116.8, 77.5), turned to -90 degrees
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Connections:
- C5 pad 1: VCC -> Net-(C5-Pad1)
- C6 pad 1: VCC -> Net-(C5-Pad1)
- J12 pad 1: unconnected-(J12-Pad1) -> GND
- J12 pad 2: unconnected-(J12-Pad2) -> GND
- J13 pad 1: Net-(J13-Pad1) -> GND
- J13 pad 9: GND -> Net-(J13-Pad9)
- J14 pad 1: unconnected-(J14-Pad1) -> GND
- J5 pad 1: Net-(J5-Pad1) -> Net-(C7-Pad1)
- J5 pad 2: Net-(J5-Pad1) -> /Alimentazione/+Vvar
- J7 pad 1: GND -> /Alimentazione/+Vvar
- J7 pad 2: GND -> /Alimentazione/+Vvar
- J7 pad 3: GND -> /Alimentazione/+Vvar
- U1 pad 2: /Alimentazione/+Vvar -> Net-(C7-Pad1)
- U10 pad 5: unconnected-(U10-Pad5) -> Net-(U10-Pad5)
- U2 pad 3: VCC -> Net-(C5-Pad1)
- U5 pad 1: Net-(J13-Pad1) -> Net-(J13-Pad2)
- U5 pad 2: Net-(J13-Pad2) -> Net-(J13-Pad3)
- U5 pad 3: Net-(J13-Pad3) -> Net-(J13-Pad4)
- U5 pad 4: Net-(J13-Pad4) -> Net-(J13-Pad5)
- U5 pad 5: Net-(J13-Pad5) -> Net-(J13-Pad6)
- U5 pad 6: Net-(J13-Pad6) -> Net-(J13-Pad7)
- U5 pad 7: Net-(J13-Pad7) -> Net-(J13-Pad8)
- U5 pad 8: Net-(J13-Pad8) -> Net-(J13-Pad9)
- U9 pad 4: unconnected-(U9-Pad4) -> Net-(U10-Pad5)
- U9 pad 5: unconnected-(U9-Pad5) -> Net-(U9-Pad5)

Commit message: Power Unit
Iniziato a sistemare l'unità alimentatore
Parts:
- added D2: VarOut, LED_THT:LED_D5.0mm, F.Cu at (16.7, 150.8)
- added D21: +5V, LED_THT:LED_D5.0mm, F.Cu at (17.0, 68.3)
- added D22: +3.3V, LED_THT:LED_D5.0mm, F.Cu at (16.8, 99.2)
- added R1: R, Resistor_THT:R_Axial_DIN0207_L6.3mm_D2.5mm_P10.16mm_Horizontal, F.Cu at (25.0, 155.8)
- added R2: R, Resistor_THT:R_Axial_DIN0207_L6.3mm_D2.5mm_P10.16mm_Horizontal, F.Cu at (-22.9, 124.4)
- added R22: R, Resistor_THT:R_Axial_DIN0207_L6.3mm_D2.5mm_P10.16mm_Horizontal, F.Cu at (-22.9, 128.5)
- added R23: R, Resistor_THT:R_Axial_DIN0207_L6.3mm_D2.5mm_P10.16mm_Horizontal, F.Cu at (24.8, 73.4)
- added R24: R, Resistor_THT:R_Axial_DIN0207_L6.3mm_D2.5mm_P10.16mm_Horizontal, F.Cu at (24.9, 104.6)
- SW1: footprint Connector_PinSocket_2.54mm:PinSocket_1x03_P2.54mm_Vertical -> Button_Switch_THT:SW_100SP1T2B4M7QE
- moved C1 219.8 mm to (40.4, 26.3), turned to 180 degrees
- moved C6 215.3 mm to (37.0, 67.1)
- moved D1 203.9 mm to (22.4, 13.2)
- moved L1 203.4 mm to (17.6, 5.23)
- moved J28 197.2 mm to (57.3, 114.9)
- moved C25 196.0 mm to (35.9, 47.0)
- moved J7 194.6 mm to (35.5, 155.2)
- moved J31 190.9 mm to (38.5, 104.6)
- moved C2 190.2 mm to (30.1, 120.6)
- moved U1 188.0 mm to (6.94, 128.3), turned to 90 degrees
- moved J32 186.9 mm to (49.5, 114.8)
- moved C5 183.7 mm to (37.0, 78.8)
- moved C23 181.8 mm to (18.7, 160.1), turned to 90 degrees
- moved C7 178.8 mm to (17.4, 141.4)
- moved C24 177.5 mm to (19.5, 89.5), turned to 90 degrees
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
Commit message: Power Supply
Seconda fase
Parts:
- added D20: 1N400x, Diode_THT:D_A-405_P10.16mm_Horizontal, F.Cu at (17.3, 75.6)
- added D3: 1n4001, Diode_THT:D_A-405_P10.16mm_Horizontal, F.Cu at (26.9, 123.2)
- added D4: 1N400x, Diode_THT:D_A-405_P10.16mm_Horizontal, F.Cu at (37.4, 64.4)
- added D5: 1n4001, Diode_THT:D_A-405_P10.16mm_Horizontal, F.Cu at (22.4, 128.6)
- added HS1: Heatsink, Heatsink2:Heatsink_28x25_Horiz, B.Cu at (32.0, 51.2)
- added HS2: Heatsink, Heatsink2:Heatsink_28x25_Horiz, B.Cu at (32.0, 110.7)
- added RV2: 5K, Potentiometer_THT:Potentiometer_Omeg_PC16BU_Vertical, B.Cu at (73.1, 149.0)
- added TP20: Potenziometer, MountingHole:MountingHole_6.5mm_Pad_Via, F.Cu at (68.0, 161.5)
- added Vmet1: 3,5_Digit_Voltmeter_3Wire, VoltmeterModule:3,5 Digit 0,28'' Voltmeter, F.Cu at (68.0, 134.4)
- C1: moved to B.Cu
- D1: value Ponte 1,5A -> D_Bridge_+AA-; footprint Diode_THT:Diode_Bridge_Round_D8.9mm -> Diode_THT:Diode_Bridge_Vishay_KBL
- Q5: value 2N3904 -> BC237
- R1: value R -> 3,3k
- R2: value R -> 240
- R22: value R -> 330k
- U1, U2: footprint Package_TO_SOT_THT:TO-220-3_Vertical -> Package_TO_SOT_THT:TO-220-3_Horizontal_TabDown; moved to B.Cu
- moved J31 73.6 mm to (-26.5, 139.2)
- moved C4 72.8 mm to (65.0, 75.1)
- moved C8 71.6 mm to (-46.0, 104.1)
- moved C9 69.8 mm to (-15.1, 96.6)
- moved Q5 64.5 mm to (21.9, 155.0), turned to 180 degrees
- moved C2 60.4 mm to (37.3, 60.7), turned to 90 degrees
- moved R22 52.9 mm to (25.5, 149.9), turned to 180 degrees
- moved C25 51.8 mm to (36.0, 98.9)
- moved J10 47.0 mm to (-9.27, 139.8)
- moved J7 45.8 mm to (-6.81, 172.7)
- moved J28 43.0 mm to (87.8, 84.7)
- moved R2 41.3 mm to (18.2, 128.7), turned to 90 degrees
- moved J32 41.1 mm to (77.1, 84.4)
- moved U2 33.8 mm to (34.6, 67.9), turned to 180 degrees
- moved U11 31.1 mm to (22.3, 89.4), turned to -90 degrees
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Connections:
- D1 pad 2: GND -> Net-(D1-Pad2)
- D1 pad 4: Net-(D1-Pad4) -> GND
- J4 pad 1: Net-(D1-Pad3) -> Net-(D1-Pad2)
- Q5 pad 1: GND -> Net-(Q5-Pad1)
- Q5 pad 3: Net-(Q5-Pad3) -> GND
- R1 pad 2: Net-(Q5-Pad3) -> Net-(Q5-Pad1)
- SW1 pad 2: Net-(D1-Pad4) -> Net-(J4-Pad2)
- SW1 pad 3: Net-(J4-Pad2) -> Net-(D1-Pad3)

Commit message: Layout Alimentatori OK
Parts:
- added F1: Polyfuse 750mA, Varistor:RV_Disc_D7mm_W5.4mm_P5mm, F.Cu at (12.3, 8.89)
- added TP21: Alimentaore Variabile, Symbol:Alimentatore Variabile, F.Cu at (43.4, 148.0)
- added TP22: Alimentatore +3,3V, Symbol:Alimentatore Variabile, F.Cu at (25.3, 106.0)
- added TP23: Alimentatore +5V, Symbol:Alimentatore Variabile, F.Cu at (25.3, 68.9)
- added TP24: Ingresso Alimentazione (7,5-15V), Symbol:Alimentatore Variabile, F.Cu at (25.3, 26.9)
- added TP25: 8 x Switch, Symbol:Alimentatore Variabile, F.Cu at (61.3, 72.2)
- added TP26: 8 x LED, Symbol:Alimentatore Variabile, F.Cu at (80.6, 30.0)
- D20, D4: value 1N400x -> 1N4001
- HS2: moved to F.Cu
- L1: value L -> 3,3mH
- R23: value R -> 680
- R24: value R -> 220
- moved C4 181.6 mm to (-85.1, -27.0)
- moved J28 181.6 mm to (-62.4, -17.4)
- moved J32 181.6 mm to (-73.1, -17.6)
- moved J8 181.6 mm to (-85.8, -13.2)
- moved D11 48.0 mm to (83.3, 25.8)
- moved D13 48.0 mm to (96.7, 25.8)
- moved TP7 48.0 mm to (96.7, 33.9)
- moved D7 48.0 mm to (56.5, 25.9)
- moved TP13 48.0 mm to (56.5, 34.0)
- moved D10 48.0 mm to (76.6, 25.8)
- moved D12 48.0 mm to (90.0, 25.8)
- moved D9 48.0 mm to (69.9, 25.8)
- moved TP10 48.0 mm to (76.6, 34.0)
- moved TP11 48.0 mm to (69.9, 34.0)
- moved D8 48.0 mm to (63.2, 25.9)
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Connections:
- J4 pad 1: Net-(D1-Pad2) -> Net-(F1-Pad1)
- TP20 pad 1: unconnected-(TP20-Pad1) -> GNDA

Commit message: Bozza con LCD 16x2
Parts:
- added DS1: HY1602E, Display:HY1602E, F.Cu at (202.8, 7.82)
- moved C21 293.6 mm to (-80.2, 114.9)
- moved J26 281.3 mm to (-119.7, 109.7)
- moved RV3 281.3 mm to (-110.7, 109.2)
- moved Uni-A4 281.3 mm to (-98.4, 109.7)
- moved *C16 252.4 mm to (-126.0, 171.5)
- moved C10 252.4 mm to (-112.5, 232.7)
- moved C17 252.4 mm to (-126.0, 176.1)
- moved C18 252.4 mm to (-115.4, 176.1)
- moved C19 252.4 mm to (-126.0, 180.8)
- moved C20 252.4 mm to (-115.4, 171.5)
- moved D6 252.4 mm to (-135.5, 140.4)
- moved J16 252.4 mm to (-115.8, 148.1)
- moved R3 252.4 mm to (-138.0, 158.2)
- moved J18 252.4 mm to (-96.4, 148.1)
- moved J22 55.0 mm to (203.6, 167.7), turned to 90 degrees
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