File: Kc/MakerLAB_r03/MakerLAB_r03.kicad_sch (KiCad schematic)
At the start: 3 parts, among them J1 Conn_01x05, J2 Conn_01x05, J3 Conn_01x05

Commit message: Bozza con LCD 16x2
Parts:
- added DS1: HY1602E, Display:HY1602E, symbol Display_Character:HY1602E
Changed lines of the file:
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@@
     (pin "5")
+  )
+  (symbol (lib_id "Display_Character:HY1602E") (at 106.68 123.825 0) (unit 1)
+    (in_bom yes) (on_board yes) (fields_autoplaced)
+    (property "Reference" "DS1" (id 0) (at 108.6994 100.33 0)
+      (effects (font (size 1.27 1.27)) (justify left))
+    )
+    (property "Value" "HY1602E" (id 1) (at 108.6994 102.87 0)
+      (effects (font (size 1.27 1.27)) (justify left))
+    )
+    (property "Footprint" "Display:HY1602E" (id 2) (at 106.68 146.685 0)
+      (effects (font (size 1.27 1.27) italic) hide)
+    )
+    (property "Datasheet" "http://www.icbank.com/data/ICBShop/board/HY1602E.pdf" (id 3) (at 111.76 121.285 0)
+      (effects (font (size 1.27 1.27)) hide)
+    )
+    (pin "1")
+    (pin "10")
+    (pin "11")
+    (pin "12")
+    (pin "13")
+    (pin "14")
+    (pin "15")
+    (pin "16")
+    (pin "2")
+    (pin "3")
+    (pin "4")
+    (pin "5")
+    (pin "6")
+    (pin "7")
+    (pin "8")
+    (pin "9")
   )
   (symbol (lib_id "Connector_Generic:Conn_01x05") (at 24.13 73.66 0) (mirror y) (unit 1)
@@
       (reference "D22") (unit 1) (value "+3.3V") (footprint "LED_THT:LED_D5.0mm")
     )
+    (path "/5ec2fb4b-6b03-4f6e-849d-4e5f1737c31d"
+      (reference "DS1") (unit 1) (value "HY1602E") (footprint "Display:HY1602E")
+    )
     (path "/fab53e88-89c0-40b1-9c44-f0dadc28ccb9/1e5a0915-6a5a-40fb-9a16-4ff4f76a5d7d"
