File: Kc/MakerLAB_r03A/MakerLAB_r03A/Visual_4Dgt.kicad_sch (KiCad schematic)
At the start: 21 parts, among them J10 Conn_01x02_Female, J11 Conn_02x10_Counter_Clockwise, J12 Conn_02x05_Counter_Clockwise, J9 Conn_02x05_Counter_Clockwise, Q1 2N3904, Q2 2N3904, Q3 2N3904, Q4 2N3904, U3 DM9368, U4 CC56-12EWA

Commit message: 27 notte
Parts:
- removed D6: LED_ALT, LED_THT:LED_D5.0mm, symbol Shield_visual4-rescue:LED_ALT-Device
- removed R3: 330, Resistor_THT:R_Axial_DIN0207_L6.3mm_D2.5mm_P10.16mm_Horizontal, symbol Device:R
Changed lines of the file:
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@@
-    (stroke (width 0) (type default) (color 0 0 0 0))
-  )
-  (wire (pts (xy 52.07 157.48) (xy 52.07 162.56))
     (stroke (width 0) (type default) (color 0 0 0 0))
   )
@@
     (stroke (width 0) (type default) (color 0 0 0 0))
   )
-  (wire (pts (xy 52.07 170.18) (xy 52.07 176.53))
-    (stroke (width 0) (type default) (color 0 0 0 0))
-  )
   (wire (pts (xy 48.26 68.58) (xy 50.8 68.58))
     (stroke (width 0) (type default) (color 0 0 0 0))
@@
   )
   (wire (pts (xy 119.38 102.87) (xy 187.96 102.87))
-    (stroke (width 0) (type default) (color 0 0 0 0))
-  )
-  (wire (pts (xy 52.07 148.59) (xy 52.07 149.86))
     (stroke (width 0) (type default) (color 0 0 0 0))
   )
@@
     )
   )
-  (symbol (lib_id "power:GND") (at 52.07 176.53 0) (unit 1)
-    (in_bom yes) (on_board yes)
-    (property "Reference" "#PWR05" (id 0) (at 52.07 182.88 0)
-      (effects (font (size 1.27 1.27)) hide)
-    )
-    (property "Value" "GND" (id 1) (at 52.197 180.9242 0))
-    (property "Footprint" "" (id 2) (at 52.07 176.53 0)
-      (effects (font (size 1.27 1.27)) hide)
-    )
-    (property "Datasheet" "" (id 3) (at 52.07 176.53 0)
-      (effects (font (size 1.27 1.27)) hide)
-    )
-    (pin "1")
-  )
   (symbol (lib_id "power:GND") (at 178.435 92.71 0) (unit 1)
     (in_bom yes) (on_board yes) (fields_autoplaced)
@@
     (pin "2")
     (pin "3")
-  )
-  (symbol (lib_id "Shield_visual4-rescue:LED_ALT-Device") (at 52.07 166.37 90) (unit 1)
-    (in_bom yes) (on_board yes)
-    (property "Reference" "D6" (id 0) (at 55.0672 165.3794 90)
-      (effects (font (size 1.27 1.27)) (justify right))
-    )
-    (property "Value" "LED_ALT" (id 1) (at 55.0672 167.6908 90)
-      (effects (font (size 1.27 1.27)) (justify right))
-    )
-    (property "Footprint" "LED_THT:LED_D5.0mm" (id 2) (at 52.07 166.37 0)
-      (effects (font (size 1.27 1.27)) hide)
-    )
-    (property "Datasheet" "~" (id 3) (at 52.07 166.37 0)
-      (effects (font (size 1.27 1.27)) hide)
-    )
-    (pin "1")
-    (pin "2")
   )
   (symbol (lib_id "power:GND") (at 39.37 156.21 0) (unit 1)
@@
     (pin "9")
   )
-  (symbol (lib_id "Device:R") (at 52.07 153.67 0) (unit 1)
-    (in_bom yes) (on_board yes)
-    (property "Reference" "R3" (id 0) (at 46.8122 153.67 90))
-    (property "Value" "330" (id 1) (at 49.1236 153.67 90))
-    (property "Footprint" "Resistor_THT:R_Axial_DIN0207_L6.3mm_D2.5mm_P10.16mm_Horizontal" (id 2) (at 50.292 153.67 90)
-      (effects (font (size 1.27 1.27)) hide)
-    )
-    (property "Datasheet" "~" (id 3) (at 52.07 153.67 0)
-      (effects (font (size 1.27 1.27)) hide)
-    )
-    (pin "1")
-    (pin "2")
-  )
   (symbol (lib_id "power:GND") (at 224.79 119.38 0) (unit 1)
