File: Kc/MakerLAB_r03A/MakerLAB_r03A/MakerLAB_r03A.kicad_pcb (KiCad board)
At the start: 2 copper layers, 374 x 178 mm, 144 parts, among them J10 Conn_01x02_Female, J11 Conn_02x10_Counter_Clockwise, J12 Conn_02x05_Counter_Clockwise, J13 GND 0 1 2 3 4 5 6 7 +5V, J14 8Bit Jumper, J15 GND 0 1 2 3 4 5 6 7 +5V, J16 Conn_02x05_Counter_Clockwise, J17 Conn_02x10_Counter_Clockwise, J18 Conn_02x05_Counter_Clockwise, J19 Conn_01x10_Female, J20 Screw_Terminal_01x02, J22 Conn_02x20_Counter_Clockwise, J23 Conn_02x20_Counter_Clockwise, J24 Conn_02x20_Counter_Clockwise, J26 Conn_01x06_Female, J28 Conn_01x03, J29 Conn_01x02_Male, J30 Conn_01x02_Male, J31 Conn_01x03, J32 Conn_01x03, J4 Barrel_Jack_MountingPin, J5 Conn_01x02_Male, J6 Conn_01x03, J7 Conn_01x03, J8 Conn_01x03, J9 Conn_02x05_Counter_Clockwise, Q1 2N3904, Q2 2N3904, Q3 2N3904, Q4 2N3904, Q5 BC237, SW1 SwGenerale, SW2 SW_DIP_x08, SW5 SW_Rotary12, U1 LM317_TO-220, U10 9368, U11 L78L33_SOT89, U2 LM7805_TO220, U3 DM9368, U4 CC56-12EWA, U5 ULN2803A, U7 NE555P, U9 9368

Commit message: 27 notte
Parts:
- removed D6: LED_ALT, LED_THT:LED_D5.0mm
- added J21: Conn_01x03, Connector_PinHeader_2.54mm:PinHeader_1x03_P2.54mm_Vertical, F.Cu at (184.4, 88.4)
- added R25: 3,3k, Resistor_THT:R_Axial_DIN0207_L6.3mm_D2.5mm_P10.16mm_Horizontal, F.Cu at (163.1, 87.2)
- added U12: HC-05, Module:XCVR_HC-05, F.Cu at (250.8, 83.9)
- LCD1: footprint Display:Adafruit_SSD1306 -> Display:TFT OLED 1.3 I2C
- R3: value 330 -> 3,3k
- moved C22 351.5 mm to (252.0, 32.7), turned to -90 degrees
- moved R3 323.6 mm to (178.1, 88.6), turned to -90 degrees
- moved C21 291.3 mm to (199.2, 32.8), turned to -90 degrees
- moved C8 229.3 mm to (177.3, 52.2)
- moved C9 97.1 mm to (79.7, 75.4), turned to -90 degrees
- moved J22 17.0 mm to (214.1, 115.4)
- moved J23 17.0 mm to (226.2, 115.5)
- moved J24 17.0 mm to (255.1, 115.4)
- moved LCD1 13.9 mm to (149.9, 86.1)
- moved R1 10.2 mm to (25.3, 154.3), turned to 180 degrees
- moved C1 7.47 mm to (38.0, 19.1)
- moved C24 6.30 mm to (23.2, 83.9), turned to 0 degrees
- moved C23 4.98 mm to (22.5, 159.3), turned to 180 degrees
- moved TP5 4.91 mm to (316.6, 88.6)
- moved Vmet1 3.04 mm to (62.4, 131.6), turned to 180 degrees
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Connections:
- LCD1 pad 1: (no net) -> VCC
- LCD1 pad 2: (no net) -> GND
- LCD1 pad 3: (no net) -> Net-(LCD1-Pad3)
- LCD1 pad 4: (no net) -> Net-(LCD1-Pad4)
- R3 pad 1: VCC -> Net-(LCD1-Pad3)
- R3 pad 2: Net-(D6-Pad2) -> VCC
Routing:
- net Net-(C16-Pad1): track 0.00 -> 175.5 mm
- net Net-(C1-Pad1): track 0.00 -> 172.6 mm
- net /Alimentazione/+Vvar: track 0.00 -> 95.3 mm
- net Net-(C24-Pad1): track 0.00 -> 84.6 mm
- net Net-(C4-Pad1): track 0.00 -> 69.6 mm
- net Net-(C7-Pad1): track 0.00 -> 63.3 mm
- net Net-(J4-Pad2): track 0.00 -> 38.3 mm
- net Net-(D1-Pad1): track 0.00 -> 37.5 mm
- net VCC: track 0.00 -> 32.3 mm
- net Net-(D2-Pad1): track 0.00 -> 23.6 mm
- net Net-(D1-Pad2): track 0.00 -> 22.8 mm
- net Net-(F1-Pad1): track 0.00 -> 12.8 mm
- net Net-(D22-Pad2): track 0.00 -> 12.1 mm
- net Net-(D21-Pad2): track 0.00 -> 10.8 mm
- net Net-(D1-Pad3): track 0.00 -> 9.83 mm
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- added copper zone on B.Cu, net GND
- added copper zone on F.Cu, net GND

Commit message: 20230328-13
20230328-13
Parts:
- added J25: IR Emitter & Sensor, Connector_PinHeader_2.54mm:PinHeader_1x03_P2.54mm_Vertical, F.Cu at (112.8, 132.8)
- added J33: Visible Light Sensor, Connector_PinHeader_2.54mm:PinHeader_1x03_P2.54mm_Vertical, F.Cu at (112.6, 156.7)
- added Q6: H21A1, Sensor:H21A1, F.Cu at (92.5, 138.4)
- added R26: 220, Resistor_THT:R_Axial_DIN0207_L6.3mm_D2.5mm_P10.16mm_Horizontal, F.Cu at (95.1, 132.9)
- added R27: 4,7k, Resistor_THT:R_Axial_DIN0207_L6.3mm_D2.5mm_P10.16mm_Horizontal, F.Cu at (97.9, 132.8)
- added R28: Left, OptoDevice:R_LDR_5.0x4.1mm_P3mm_Vertical, F.Cu at (84.5, 167.4)
- added R29: Right, OptoDevice:R_LDR_5.0x4.1mm_P3mm_Vertical, F.Cu at (109.4, 167.4)
- added R30: 33k, Resistor_THT:R_Axial_DIN0207_L6.3mm_D2.5mm_P10.16mm_Horizontal, F.Cu at (94.0, 157.0)
- added R31: Mono, OptoDevice:R_LDR_5.0x4.1mm_P3mm_Vertical, F.Cu at (97.3, 167.4)
- added TP30: Pulse Generator, SerigrafieMakerLAB:Clock NE555, F.Cu at (98.7, 133.1)
- U12: value HC-05 -> HC-05 (ZC142200); footprint Module:XCVR_HC-05 -> RF_Module:HC-05 Module Horizontal (ZC14200)
- moved TP29 237.3 mm to (-138.4, 126.6)
- moved J17 79.5 mm to (178.5, 135.2), turned to 0 degrees
- moved J26 77.4 mm to (181.0, 159.4), turned to 180 degrees
- moved J24 65.3 mm to (209.6, 162.3), turned to 180 degrees
- moved J22 59.4 mm to (250.6, 162.3), turned to 180 degrees
- moved J23 48.3 mm to (238.5, 162.2), turned to 180 degrees
- moved R15 46.7 mm to (174.0, 167.5), turned to 180 degrees
- moved C17 30.5 mm to (165.0, 147.2), turned to 0 degrees
- moved D17 26.5 mm to (122.2, 114.5)
- moved R17 18.1 mm to (130.9, 167.4)
- moved U7 16.8 mm to (121.7, 157.0)
- moved U12 13.8 mm to (237.3, 87.1), turned to 180 degrees
- moved R25 12.7 mm to (175.1, 83.1), turned to 90 degrees
- moved R16 12.4 mm to (174.0, 163.0), turned to 180 degrees
- moved C18 9.39 mm to (129.2, 162.0)
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