File: Kc/MakerLAB_r03A/MakerLAB_r03A/MakerLAB_r03A.kicad_sch (KiCad schematic)
At the start: 3 parts, among them J1 Conn_01x05, J2 Conn_01x05, J3 Conn_01x05

Commit message: 27 notte
Parts:
- added U12: HC-05, XCVR_HC-05, symbol MCU_Module:HC-05
Connections:
- new net: U12.13 (GND), U12.21 (GND), U12.22 (GND)
Changed lines of the file:
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@@
     (pin "5")
+  )
+  (symbol (lib_id "MCU_Module:HC-05") (at 62.865 153.67 0) (unit 1)
+    (in_bom yes) (on_board yes) (fields_autoplaced)
+    (property "Reference" "U12" (id 0) (at 62.865 118.11 0))
+    (property "Value" "HC-05" (id 1) (at 62.865 120.65 0))
+    (property "Footprint" "XCVR_HC-05" (id 2) (at 62.865 153.67 0)
+      (effects (font (size 1.27 1.27)) (justify bottom) hide)
+    )
+    (property "Datasheet" "" (id 3) (at 62.865 153.67 0)
+      (effects (font (size 1.27 1.27)) hide)
+    )
+    (property "PARTREV" "v1.0" (id 4) (at 62.865 153.67 0)
+      (effects (font (size 1.27 1.27)) (justify bottom) hide)
+    )
+    (property "STANDARD" "Manufacturer Recommendations" (id 5) (at 62.865 153.67 0)
+      (effects (font (size 1.27 1.27)) (justify bottom) hide)
+    )
+    (property "MF" "HuiCheng" (id 6) (at 62.865 153.67 0)
+      (effects (font (size 1.27 1.27)) (justify bottom) hide)
+    )
+    (pin "1")
+    (pin "10")
+    (pin "11")
+    (pin "12")
+    (pin "13")
+    (pin "15")
+    (pin "16")
+    (pin "17")
+    (pin "18")
+    (pin "19")
+    (pin "2")
+    (pin "20")
+    (pin "21")
+    (pin "22")
+    (pin "23")
+    (pin "24")
+    (pin "25")
+    (pin "26")
+    (pin "27")
+    (pin "28")
+    (pin "29")
+    (pin "3")
+    (pin "30")
+    (pin "31")
+    (pin "32")
+    (pin "33")
+    (pin "34")
+    (pin "4")
+    (pin "5")
+    (pin "6")
+    (pin "7")
+    (pin "8")
+    (pin "9")
   )
   (sheet (at 102.87 63.5) (size 16.51 13.97) (fields_autoplaced)
@@
       (reference "#PWR04") (unit 1) (value "+5V") (footprint "")
     )
-    (path "/3fdafdb4-8fb2-4faf-beb8-83b0478cdff5/96e4e0b2-0c64-4a5a-bff6-1119e353840a"
-      (reference "#PWR05") (unit 1) (value "GND") (footprint "")
-    )
     (path "/3fdafdb4-8fb2-4faf-beb8-83b0478cdff5/02ed7423-c3d9-49be-8e1e-327aba76b89c"
       (reference "#PWR06") (unit 1) (value "+5V") (footprint "")
@@
       (reference "D5") (unit 1) (value "1n4001") (footprint "Diode_THT:D_A-405_P10.16mm_Horizontal")
     )
-    (path "/3fdafdb4-8fb2-4faf-beb8-83b0478cdff5/ad4a3c25-9bc4-4b63-a0f0-7d308a076c49"
-      (reference "D6") (unit 1) (value "LED_ALT") (footprint "LED_THT:LED_D5.0mm")
-    )
     (path "/84edcc0d-58f3-4926-bbd5-9d9520a90734/01f3f89b-14d8-4e79-8e31-70c0b46ceb23"
       (reference "D7") (unit 1) (value "7") (footprint "LED_THT:LED_D5.0mm")
@@
       (reference "J20") (unit 1) (value "Screw_Terminal_01x02") (footprint "TerminalBlock:TerminalBlock_bornier-2_P5.08mm")
     )
+    (path "/936db2ac-1acd-4015-81fa-2968def21830/b0aa2193-5bdd-4e15-8d70-5a6071e29b46"
+      (reference "J21") (unit 1) (value "Conn_01x03") (footprint "Connector_PinHeader_2.54mm:PinHeader_1x03_P2.54mm_Vertical")
+    )
     (path "/4655614b-d320-4698-a75c-caa6a671ceee/30d53521-c628-42bd-96b5-44e68b7948c2"
       (reference "J22") (unit 1) (value "Conn_02x20_Counter_Clockwise") (footprint "Connector_PinSocket_2.54mm:PinSocket_2x20_P2.54mm_Vertical")
@@
     )
     (path "/936db2ac-1acd-4015-81fa-2968def21830/f2660a19-eccb-4c2b-9166-2f1a28e62ef1"
-      (reference "LCD1") (unit 1) (value "SSD1306_OLED128x64_I2C") (footprint "Display:Adafruit_SSD1306")
+      (reference "LCD1") (unit 1) (value "SSD1306_OLED128x64_I2C") (footprint "Display:TFT OLED 1.3 I2C")
     )
     (path "/3fdafdb4-8fb2-4faf-beb8-83b0478cdff5/e797b41f-9826-472e-af49-3a8d1cd7098a"
@@
       (reference "R2") (unit 1) (value "240") (footprint "Resistor_THT:R_Axial_DIN0207_L6.3mm_D2.5mm_P10.16mm_Horizontal")
     )
-    (path "/3fdafdb4-8fb2-4faf-beb8-83b0478cdff5/f64ce6cd-013a-496d-afc7-e16f5b2ef7b9"
-      (reference "R3") (unit 1) (value "330") (footprint "Resistor_THT:R_Axial_DIN0207_L6.3mm_D2.5mm_P10.16mm_Horizontal")
+    (path "/936db2ac-1acd-4015-81fa-2968def21830/70acf039-5b0b-4562-ac5b-9698c55dbd28"
+      (reference "R3") (unit 1) (value "3,3k") (footprint "Resistor_THT:R_Axial_DIN0207_L6.3mm_D2.5mm_P10.16mm_Horizontal")
     )
     (path "/3fdafdb4-8fb2-4faf-beb8-83b0478cdff5/c7807945-7702-4701-ae9a-fdd3c32f0f94"
@@
       (reference "R24") (unit 1) (value "220") (footprint "Resistor_THT:R_Axial_DIN0207_L6.3mm_D2.5mm_P10.16mm_Horizontal")
     )
+    (path "/936db2ac-1acd-4015-81fa-2968def21830/7363fb1f-c868-4438-93e6-e02a892616d6"
+      (reference "R25") (unit 1) (value "3,3k") (footprint "Resistor_THT:R_Axial_DIN0207_L6.3mm_D2.5mm_P10.16mm_Horizontal")
+    )
     (path "/84edcc0d-58f3-4926-bbd5-9d9520a90734/2b35632c-b8b2-4fba-8fc1-5127f843232f"
       (reference "RN1") (unit 1) (value "Resistor Array") (footprint "Package_DIP:DIP-16_W7.62mm_Socket_LongPads")
@@
       (reference "TP29") (unit 1) (value "8 x LED") (footprint "SerigrafieMakerLAB:Clock NE555")
     )
+    (path "/1c7b6ba1-9bc1-4836-88a5-b185a760b165/df6c0773-6376-4e47-b98b-9de65ed6dc0a"
+      (reference "TP30") (unit 1) (value "2x7Segment") (footprint "SerigrafieMakerLAB:Clock NE555")
+    )
     (path "/fab53e88-89c0-40b1-9c44-f0dadc28ccb9/c5a00fd2-4cd0-429e-9a6d-bd151e0d6d4f"
       (reference "U1") (unit 1) (value "LM317_TO-220") (footprint "Package_TO_SOT_THT:TO-220-3_Horizontal_TabDown")
@@
       (reference "U11") (unit 1) (value "L78L33_SOT89") (footprint "Package_TO_SOT_SMD:SOT-223")
     )
+    (path "/bd4954c1-3488-46fe-82c7-92d55c68f922"
+      (reference "U12") (unit 1) (value "HC-05") (footprint "XCVR_HC-05")
+    )
     (path "/7b083e6b-8037-4945-a6a7-d033f55692d8/e5dec7fc-12c8-4cdc-be25-c2ebc298277a"

Commit message: 20230328-13
20230328-13
Parts:
- removed U12: HC-05, XCVR_HC-05, symbol MCU_Module:HC-05
Other:
- added sheet BT to Serial (BTtoSerial.kicad_sch)
- added sheet IR Sensor (IRSensor.kicad_sch)
- added sheet Photoresistor (Photoresistor.kicad_sch)
Changed lines of the file:
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@@
     (pin "5")
-  )
-  (symbol (lib_id "MCU_Module:HC-05") (at 62.865 153.67 0) (unit 1)
-    (in_bom yes) (on_board yes) (fields_autoplaced)
-    (property "Reference" "U12" (id 0) (at 62.865 118.11 0))
-    (property "Value" "HC-05" (id 1) (at 62.865 120.65 0))
-    (property "Footprint" "XCVR_HC-05" (id 2) (at 62.865 153.67 0)
-      (effects (font (size 1.27 1.27)) (justify bottom) hide)
-    )
-    (property "Datasheet" "" (id 3) (at 62.865 153.67 0)
-      (effects (font (size 1.27 1.27)) hide)
-    )
-    (property "PARTREV" "v1.0" (id 4) (at 62.865 153.67 0)
-      (effects (font (size 1.27 1.27)) (justify bottom) hide)
-    )
-    (property "STANDARD" "Manufacturer Recommendations" (id 5) (at 62.865 153.67 0)
-      (effects (font (size 1.27 1.27)) (justify bottom) hide)
-    )
-    (property "MF" "HuiCheng" (id 6) (at 62.865 153.67 0)
-      (effects (font (size 1.27 1.27)) (justify bottom) hide)
-    )
-    (pin "1")
-    (pin "10")
-    (pin "11")
-    (pin "12")
-    (pin "13")
-    (pin "15")
-    (pin "16")
-    (pin "17")
-    (pin "18")
-    (pin "19")
-    (pin "2")
-    (pin "20")
-    (pin "21")
-    (pin "22")
-    (pin "23")
-    (pin "24")
-    (pin "25")
-    (pin "26")
-    (pin "27")
-    (pin "28")
-    (pin "29")
-    (pin "3")
-    (pin "30")
-    (pin "31")
-    (pin "32")
-    (pin "33")
-    (pin "34")
-    (pin "4")
-    (pin "5")
-    (pin "6")
-    (pin "7")
-    (pin "8")
-    (pin "9")
   )
   (sheet (at 102.87 63.5) (size 16.51 13.97) (fields_autoplaced)
@@
     )
   )
+  (sheet (at 149.86 123.19) (size 46.99 29.21) (fields_autoplaced)
+    (stroke (width 0.1524) (type solid) (color 0 0 0 0))
+    (fill (color 0 0 0 0.0000))
+    (property "Sheet name" "IR Sensor" (id 0) (at 149.86 122.4784 0)
+      (effects (font (size 1.27 1.27)) (justify left bottom))
+    )
+    (property "Sheet file" "IRSensor.kicad_sch" (id 1) (at 149.86 152.9846 0)
+      (effects (font (size 1.27 1.27)) (justify left top))
+    )
+  )
   (sheet (at 54.61 20.32) (size 31.75 11.43) (fields_autoplaced)
     (stroke (width 0.1524) (type solid) (color 0 0 0 0))
@@
     (pin "+5V" input (at 144.78 41.91 180)
       (effects (font (size 1.27 1.27)) (justify left))
+    )
+  )
+  (sheet (at 208.28 97.79) (size 38.1 25.4) (fields_autoplaced)
+    (stroke (width 0.1524) (type solid) (color 0 0 0 0))
+    (fill (color 0 0 0 0.0000))
+    (property "Sheet name" "Photoresistor" (id 0) (at 208.28 97.0784 0)
+      (effects (font (size 1.27 1.27)) (justify left bottom))
+    )
+    (property "Sheet file" "Photoresistor.kicad_sch" (id 1) (at 208.28 123.7746 0)
+      (effects (font (size 1.27 1.27)) (justify left top))
     )
   )
@@
     (pin "GNG_pwr" input (at 55.88 72.39 180)
       (effects (font (size 1.27 1.27)) (justify left))
+    )
+  )
+  (sheet (at 44.45 129.54) (size 63.5 33.02) (fields_autoplaced)
+    (stroke (width 0.1524) (type solid) (color 0 0 0 0))
+    (fill (color 0 0 0 0.0000))
+    (property "Sheet name" "BT to Serial" (id 0) (at 44.45 128.8284 0)
+      (effects (font (size 1.27 1.27)) (justify left bottom))
+    )
+    (property "Sheet file" "BTtoSerial.kicad_sch" (id 1) (at 44.45 163.1446 0)
+      (effects (font (size 1.27 1.27)) (justify left top))
     )
   )
@@
     (path "/1c7b6ba1-9bc1-4836-88a5-b185a760b165" (page "12"))
     (path "/936db2ac-1acd-4015-81fa-2968def21830" (page "13"))
+    (path "/2e13182b-77d9-4e81-a15f-ca823b99bb6c" (page "14"))
+    (path "/79ad9125-782d-43b3-829f-b6bbdd2a310f" (page "15"))
+    (path "/90cb1aeb-5b36-4bf9-b4a8-315430d66e7b" (page "16"))
   )
   (symbol_instances
@@
       (reference "#PWR0109") (unit 1) (value "GND") (footprint "")
     )
+    (path "/2e13182b-77d9-4e81-a15f-ca823b99bb6c/128609a3-aa7b-44a0-97a6-a3555e2518a7"
+      (reference "#PWR0110") (unit 1) (value "GND") (footprint "")
+    )
+    (path "/2e13182b-77d9-4e81-a15f-ca823b99bb6c/89a5039f-74e5-4334-a325-cdb99956c5a7"
+      (reference "#PWR0111") (unit 1) (value "GND") (footprint "")
+    )
     (path "/62ab733d-ee67-4f7c-8a1e-1b8f9ec01131/48986c64-6854-480d-9593-dd61075c74a0"
       (reference "*C16") (unit 1) (value "330pF") (footprint "Capacitor_THT:C_Axial_L5.1mm_D3.1mm_P7.50mm_Horizontal")
@@
       (reference "J24") (unit 1) (value "Conn_02x20_Counter_Clockwise") (footprint "Connector_PinSocket_2.54mm:PinSocket_2x20_P2.54mm_Vertical")
     )
+    (path "/2e13182b-77d9-4e81-a15f-ca823b99bb6c/a1b790d3-9aac-47aa-a67b-12fa67c1db1a"
+      (reference "J25") (unit 1) (value "IR Emitter & Sensor") (footprint "Connector_PinHeader_2.54mm:PinHeader_1x03_P2.54mm_Vertical")
+    )
     (path "/62ab733d-ee67-4f7c-8a1e-1b8f9ec01131/0f244bee-5da1-4d0b-9853-8facd5b0ed9c"
       (reference "J26") (unit 1) (value "Conn_01x06_Female") (footprint "Connector_PinHeader_2.54mm:PinHeader_1x06_P2.54mm_Vertical")
@@
       (reference "J32") (unit 1) (value "Conn_01x03") (footprint "Connector_PinHeader_2.54mm:PinHeader_1x03_P2.54mm_Vertical")
     )
+    (path "/79ad9125-782d-43b3-829f-b6bbdd2a310f/f7203bf7-332f-41c5-aa2f-bbaf6dc3c4a6"
+      (reference "J33") (unit 1) (value "Visible Light Sensor") (footprint "Connector_PinHeader_2.54mm:PinHeader_1x03_P2.54mm_Vertical")
+    )
     (path "/fab53e88-89c0-40b1-9c44-f0dadc28ccb9/d1d6b82f-d413-4020-a4d1-e737d99f4b24"
       (reference "L1") (unit 1) (value "3,3mH") (footprint "Inductor_THT:L_Axial_L12.0mm_D5.0mm_P15.24mm_Horizontal_Fastron_MISC")
@@
       (reference "Q5") (unit 1) (value "BC237") (footprint "Package_TO_SOT_THT:TO-92_Inline")
     )
+    (path "/2e13182b-77d9-4e81-a15f-ca823b99bb6c/00cec69a-d9a9-4880-9b5f-ed6f47a9aa15"
+      (reference "Q6") (unit 1) (value "H21A1") (footprint "Sensor:H21A1")
+    )
     (path "/fab53e88-89c0-40b1-9c44-f0dadc28ccb9/6ff181c9-b25a-46e0-b627-21bc1b1eacea"
       (reference "R1") (unit 1) (value "3,3k") (footprint "Resistor_THT:R_Axial_DIN0207_L6.3mm_D2.5mm_P10.16mm_Horizontal")
@@
       (reference "R25") (unit 1) (value "3,3k") (footprint "Resistor_THT:R_Axial_DIN0207_L6.3mm_D2.5mm_P10.16mm_Horizontal")
     )
+    (path "/2e13182b-77d9-4e81-a15f-ca823b99bb6c/5c694ffb-48d7-4d44-8a26-25343de389d2"
+      (reference "R26") (unit 1) (value "220") (footprint "Resistor_THT:R_Axial_DIN0207_L6.3mm_D2.5mm_P10.16mm_Horizontal")
+    )
+    (path "/2e13182b-77d9-4e81-a15f-ca823b99bb6c/0a1a539a-cfc8-4353-a323-c56330107479"
+      (reference "R27") (unit 1) (value "4,7k") (footprint "Resistor_THT:R_Axial_DIN0207_L6.3mm_D2.5mm_P10.16mm_Horizontal")
+    )
+    (path "/79ad9125-782d-43b3-829f-b6bbdd2a310f/9547c787-e780-4303-914a-465b22ca1b57"
+      (reference "R28") (unit 1) (value "Left") (footprint "OptoDevice:R_LDR_5.0x4.1mm_P3mm_Vertical")
+    )
+    (path "/79ad9125-782d-43b3-829f-b6bbdd2a310f/7fb4ab74-ba57-417c-9a00-2eb4e7008cfc"
+      (reference "R29") (unit 1) (value "Right") (footprint "OptoDevice:R_LDR_5.0x4.1mm_P3mm_Vertical")
+    )
+    (path "/79ad9125-782d-43b3-829f-b6bbdd2a310f/caed2325-6f65-4c6c-ace7-6a283f755bb2"
+      (reference "R30") (unit 1) (value "33k") (footprint "Resistor_THT:R_Axial_DIN0207_L6.3mm_D2.5mm_P10.16mm_Horizontal")
+    )
+    (path "/79ad9125-782d-43b3-829f-b6bbdd2a310f/aefaed44-0140-4a91-b146-29f3c702ad59"
+      (reference "R31") (unit 1) (value "Mono") (footprint "OptoDevice:R_LDR_5.0x4.1mm_P3mm_Vertical")
+    )
     (path "/84edcc0d-58f3-4926-bbd5-9d9520a90734/2b35632c-b8b2-4fba-8fc1-5127f843232f"
       (reference "RN1") (unit 1) (value "Resistor Array") (footprint "Package_DIP:DIP-16_W7.62mm_Socket_LongPads")
@@
     )
     (path "/1c7b6ba1-9bc1-4836-88a5-b185a760b165/df6c0773-6376-4e47-b98b-9de65ed6dc0a"
-      (reference "TP30") (unit 1) (value "2x7Segment") (footprint "SerigrafieMakerLAB:Clock NE555")
+      (reference "TP30") (unit 1) (value "Pulse Generator") (footprint "SerigrafieMakerLAB:Clock NE555")
     )
     (path "/fab53e88-89c0-40b1-9c44-f0dadc28ccb9/c5a00fd2-4cd0-429e-9a6d-bd151e0d6d4f"
@@
       (reference "U11") (unit 1) (value "L78L33_SOT89") (footprint "Package_TO_SOT_SMD:SOT-223")
     )
-    (path "/bd4954c1-3488-46fe-82c7-92d55c68f922"
-      (reference "U12") (unit 1) (value "HC-05") (footprint "XCVR_HC-05")
+    (path "/90cb1aeb-5b36-4bf9-b4a8-315430d66e7b/b02cd71e-b7e5-4eed-89af-28e2fad49650"
+      (reference "U12") (unit 1) (value "HC-05 (ZC142200)") (footprint "RF_Module:HC-05 Module Horizontal (ZC14200)")
     )
     (path "/7b083e6b-8037-4945-a6a7-d033f55692d8/e5dec7fc-12c8-4cdc-be25-c2ebc298277a"
