File: Kc/MakerLAB_r03A/MakerLAB_r03A/OLED_128x64.kicad_sch (KiCad schematic)
At the start: 1 part

Commit message: 27 notte
Parts:
- added J21: Conn_01x03, Connector_PinHeader_2.54mm:PinHeader_1x03_P2.54mm_Vertical, symbol Connector_Generic:Conn_01x03
- added R25, R3: 3,3k, Resistor_THT:R_Axial_DIN0207_L6.3mm_D2.5mm_P10.16mm_Horizontal, symbol Device:R
- LCD1: footprint Display:Adafruit_SSD1306 -> Display:TFT OLED 1.3 I2C
Connections:
- net GND: now also LCD1.2 (GND), J21.1 (Pin_1); no longer LCD1. (Vcc)
- net VCC: now also LCD1.1 (Vcc), R25.2, R3.2; no longer LCD1. (Vcc)
- removed net OLED_SCL: LCD1. (Vcc)
- removed net OLED_SDA: LCD1. (Vcc)
- new net: J21.2 (Pin_2), LCD1.3 (SCL), R3.1
- new net: J21.3 (Pin_3), LCD1.4 (SDA), R25.1
Changed lines of the file:
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@@
 (kicad_sch (version 20211123) (generator eeschema)
   (paper "A4")
+  (junction (at 167.64 74.295) (diameter 0) (color 0 0 0 0)
+  )
+  (junction (at 144.78 83.82) (diameter 0) (color 0 0 0 0)
+  )
+  (junction (at 167.64 64.77) (diameter 0) (color 0 0 0 0)
+  )
+  (junction (at 129.54 87.63) (diameter 0) (color 0 0 0 0)
+  )
+  (junction (at 139.7 74.295) (diameter 0) (color 0 0 0 0)
+  )
   (wire (pts (xy 144.78 83.82) (xy 144.78 92.71))
+    (stroke (width 0) (type default) (color 0 0 0 0))
+  )
+  (wire (pts (xy 164.465 83.82) (xy 167.64 83.82))
+    (stroke (width 0) (type default) (color 0 0 0 0))
+  )
+  (wire (pts (xy 144.78 69.215) (xy 144.78 83.82))
+    (stroke (width 0) (type default) (color 0 0 0 0))
+  )
+  (wire (pts (xy 167.64 74.295) (xy 167.64 83.82))
     (stroke (width 0) (type default) (color 0 0 0 0))
   )
@@
     (stroke (width 0) (type default) (color 0 0 0 0))
   )
+  (wire (pts (xy 167.64 53.34) (xy 167.64 64.77))
+    (stroke (width 0) (type default) (color 0 0 0 0))
+  )
+  (wire (pts (xy 139.7 69.215) (xy 144.78 69.215))
+    (stroke (width 0) (type default) (color 0 0 0 0))
+  )
+  (wire (pts (xy 134.62 57.15) (xy 134.62 60.325))
+    (stroke (width 0) (type default) (color 0 0 0 0))
+  )
   (wire (pts (xy 129.54 92.71) (xy 129.54 87.63))
     (stroke (width 0) (type default) (color 0 0 0 0))
   )
-  (wire (pts (xy 139.7 83.82) (xy 139.7 92.71))
+  (wire (pts (xy 139.7 74.295) (xy 139.7 92.71))
     (stroke (width 0) (type default) (color 0 0 0 0))
   )
-  (wire (pts (xy 134.62 81.28) (xy 134.62 92.71))
+  (wire (pts (xy 137.16 57.15) (xy 137.16 74.295))
+    (stroke (width 0) (type default) (color 0 0 0 0))
+  )
+  (wire (pts (xy 129.54 60.325) (xy 129.54 87.63))
+    (stroke (width 0) (type default) (color 0 0 0 0))
+  )
+  (wire (pts (xy 134.62 64.77) (xy 167.64 64.77))
+    (stroke (width 0) (type default) (color 0 0 0 0))
+  )
+  (wire (pts (xy 134.62 64.77) (xy 134.62 92.71))
+    (stroke (width 0) (type default) (color 0 0 0 0))
+  )
+  (wire (pts (xy 139.7 74.295) (xy 156.845 74.295))
     (stroke (width 0) (type default) (color 0 0 0 0))
   )
@@
     (stroke (width 0) (type default) (color 0 0 0 0))
   )
-  (hierarchical_label "OLED_SCL" (shape input) (at 139.7 83.82 90)
-    (effects (font (size 1.27 1.27)) (justify left))
+  (wire (pts (xy 164.465 74.295) (xy 167.64 74.295))
+    (stroke (width 0) (type default) (color 0 0 0 0))
   )
-  (hierarchical_label "OLED_SDA" (shape input) (at 144.78 83.82 90)
-    (effects (font (size 1.27 1.27)) (justify left))
+  (wire (pts (xy 137.16 74.295) (xy 139.7 74.295))
+    (stroke (width 0) (type default) (color 0 0 0 0))
   )
-  (symbol (lib_id "power:VCC") (at 134.62 81.28 0) (unit 1)
+  (wire (pts (xy 134.62 60.325) (xy 129.54 60.325))
+    (stroke (width 0) (type default) (color 0 0 0 0))
+  )
+  (wire (pts (xy 139.7 57.15) (xy 139.7 69.215))
+    (stroke (width 0) (type default) (color 0 0 0 0))
+  )
+  (wire (pts (xy 167.64 64.77) (xy 167.64 74.295))
+    (stroke (width 0) (type default) (color 0 0 0 0))
+  )
+  (wire (pts (xy 144.78 83.82) (xy 156.845 83.82))
+    (stroke (width 0) (type default) (color 0 0 0 0))
+  )
+  (symbol (lib_id "Device:R") (at 160.655 74.295 90) (unit 1)
     (in_bom yes) (on_board yes) (fields_autoplaced)
-    (property "Reference" "#PWR0108" (id 0) (at 134.62 85.09 0)
+    (property "Reference" "R3" (id 0) (at 160.655 67.945 90))
+    (property "Value" "3,3k" (id 1) (at 160.655 70.485 90))
+    (property "Footprint" "Resistor_THT:R_Axial_DIN0207_L6.3mm_D2.5mm_P10.16mm_Horizontal" (id 2) (at 160.655 76.073 90)
       (effects (font (size 1.27 1.27)) hide)
     )
-    (property "Value" "VCC" (id 1) (at 134.62 76.2 0))
-    (property "Footprint" "" (id 2) (at 134.62 81.28 0)
-      (effects (font (size 1.27 1.27)) hide)
-    )
-    (property "Datasheet" "" (id 3) (at 134.62 81.28 0)
+    (property "Datasheet" "~" (id 3) (at 160.655 74.295 0)
       (effects (font (size 1.27 1.27)) hide)
     )
     (pin "1")
+    (pin "2")
+  )
+  (symbol (lib_id "Device:R") (at 160.655 83.82 90) (unit 1)
+    (in_bom yes) (on_board yes) (fields_autoplaced)
+    (property "Reference" "R25" (id 0) (at 160.655 77.47 90))
+    (property "Value" "3,3k" (id 1) (at 160.655 80.01 90))
+    (property "Footprint" "Resistor_THT:R_Axial_DIN0207_L6.3mm_D2.5mm_P10.16mm_Horizontal" (id 2) (at 160.655 85.598 90)
+      (effects (font (size 1.27 1.27)) hide)
+    )
+    (property "Datasheet" "~" (id 3) (at 160.655 83.82 0)
+      (effects (font (size 1.27 1.27)) hide)
+    )
+    (pin "1")
+    (pin "2")
+  )
+  (symbol (lib_id "power:VCC") (at 167.64 53.34 0) (unit 1)
+    (in_bom yes) (on_board yes) (fields_autoplaced)
+    (property "Reference" "#PWR0108" (id 0) (at 167.64 57.15 0)
+      (effects (font (size 1.27 1.27)) hide)
+    )
+    (property "Value" "VCC" (id 1) (at 167.64 48.26 0))
+    (property "Footprint" "" (id 2) (at 167.64 53.34 0)
+      (effects (font (size 1.27 1.27)) hide)
+    )
+    (property "Datasheet" "" (id 3) (at 167.64 53.34 0)
+      (effects (font (size 1.27 1.27)) hide)
+    )
+    (pin "1")
+  )
+  (symbol (lib_id "Connector_Generic:Conn_01x03") (at 137.16 52.07 90) (unit 1)
+    (in_bom yes) (on_board yes) (fields_autoplaced)
+    (property "Reference" "J21" (id 0) (at 142.24 50.7999 90)
+      (effects (font (size 1.27 1.27)) (justify right))
+    )
+    (property "Value" "Conn_01x03" (id 1) (at 142.24 53.3399 90)
+      (effects (font (size 1.27 1.27)) (justify right))
+    )
+    (property "Footprint" "Connector_PinHeader_2.54mm:PinHeader_1x03_P2.54mm_Vertical" (id 2) (at 137.16 52.07 0)
+      (effects (font (size 1.27 1.27)) hide)
+    )
+    (property "Datasheet" "~" (id 3) (at 137.16 52.07 0)
+      (effects (font (size 1.27 1.27)) hide)
+    )
+    (pin "1")
+    (pin "2")
+    (pin "3")
   )
   (symbol (lib_id "power:GND") (at 113.03 95.25 0) (unit 1)
@@
       (effects (font (size 1.27 1.27)) (justify left))
     )
-    (property "Footprint" "Display:Adafruit_SSD1306" (id 2) (at 137.16 102.87 0)
+    (property "Footprint" "Display:TFT OLED 1.3 I2C" (id 2) (at 137.16 102.87 0)
       (effects (font (size 1.27 1.27)) hide)
     )
@@
       (effects (font (size 1.27 1.27)) hide)
     )
-    (pin "")
-    (pin "")
-    (pin "")
-    (pin "")
+    (pin "2")
+    (pin "3")
+    (pin "4")
+    (pin "1")
   )
 )
