File: Kc/MakerLAB_r03A/MakerLAB_r03A/PadSerigrafie.kicad_sch (KiCad schematic)
At the start: 15 parts

Commit message: 27 notte
Parts:
- added TP30: 2x7Segment, SerigrafieMakerLAB:Clock NE555, symbol Connector:TestPoint
Changed lines of the file:
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@@
+    (pin "1")
+  )
+  (symbol (lib_id "Connector:TestPoint") (at 142.24 116.84 0) (unit 1)
+    (in_bom yes) (on_board yes) (fields_autoplaced)
+    (property "Reference" "TP30" (id 0) (at 144.78 112.2679 0)
+      (effects (font (size 1.27 1.27)) (justify left))
+    )
+    (property "Value" "2x7Segment" (id 1) (at 144.78 114.8079 0)
+      (effects (font (size 1.27 1.27)) (justify left))
+    )
+    (property "Footprint" "SerigrafieMakerLAB:Clock NE555" (id 2) (at 147.32 116.84 0)
+      (effects (font (size 1.27 1.27)) hide)
+    )
+    (property "Datasheet" "~" (id 3) (at 147.32 116.84 0)
+      (effects (font (size 1.27 1.27)) hide)
+    )
     (pin "1")
   )

Commit message: 20230328-13
20230328-13
Parts:
- TP30: value 2x7Segment -> Pulse Generator
Changed lines of the file:
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@@
       (effects (font (size 1.27 1.27)) (justify left))
     )
-    (property "Value" "2x7Segment" (id 1) (at 144.78 114.8079 0)
+    (property "Value" "Pulse Generator" (id 1) (at 144.78 114.8079 0)
       (effects (font (size 1.27 1.27)) (justify left))
     )
