File: Kc/MakerLAB_r03B/Gen_Clock.kicad_sch (KiCad schematic)
At the start: 16 parts, among them J17 Conn_02x10_Counter_Clockwise, J26 Conn_01x06_Female, SW5 SW_Rotary12, U7 NE555P

Commit message: versione r03B della notte del 28 marzo 2023
Connections:
- net Clock: no longer names the net of D17.1 (K), J17.14 (Pin_14), J17.15 (Pin_15), J17.16 (Pin_16), J17.17 (Pin_17), J17.4 (Pin_4), J17.5 (Pin_5), J17.6 (Pin_6), J17.7 (Pin_7), U7.3 (Q)
Changed lines of the file:
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@@
   (junction (at 64.77 39.37) (diameter 0) (color 0 0 0 0)
   )
-  (junction (at 147.32 55.88) (diameter 0) (color 0 0 0 0)
-  )
   (junction (at 120.65 114.3) (diameter 0) (color 0 0 0 0)
   )
@@
   )
   (wire (pts (xy 140.97 44.45) (xy 140.97 55.88))
-    (stroke (width 0) (type default) (color 0 0 0 0))
-  )
-  (wire (pts (xy 147.32 55.88) (xy 149.86 55.88))
     (stroke (width 0) (type default) (color 0 0 0 0))
   )
@@
     (effects (font (size 1.27 1.27)) (justify left))
   )
-  (hierarchical_label "Clock" (shape output) (at 149.86 55.88 0)
-    (effects (font (size 1.27 1.27)) (justify left))
-  )
