File: Kc/MakerLAB_r03B/Input_8bit.kicad_sch (KiCad schematic)
At the start: 3 parts, among them J15 GND 0 1 2 3 4 5 6 7 +5V, SW2 SW_DIP_x08

Commit message: versione r03B della notte del 28 marzo 2023
Changed lines of the file:
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@@
   (junction (at 143.51 78.74) (diameter 0) (color 0 0 0 0)
+  )
+  (junction (at 165.1 60.96) (diameter 0) (color 0 0 0 0)
   )
   (junction (at 156.21 91.44) (diameter 0) (color 0 0 0 0)
@@
   )
   (junction (at 153.67 88.9) (diameter 0) (color 0 0 0 0)
-  )
-  (junction (at 165.1 76.2) (diameter 0) (color 0 0 0 0)
   )
   (junction (at 146.05 60.96) (diameter 0) (color 0 0 0 0)
@@
   )
   (wire (pts (xy 124.46 101.6) (xy 160.02 101.6))
+    (stroke (width 0) (type default) (color 0 0 0 0))
+  )
+  (wire (pts (xy 165.1 60.96) (xy 165.1 53.975))
     (stroke (width 0) (type default) (color 0 0 0 0))
   )
@@
     (stroke (width 0) (type default) (color 0 0 0 0))
   )
-  (wire (pts (xy 165.1 76.2) (xy 165.1 104.14))
-    (stroke (width 0) (type default) (color 0 0 0 0))
-  )
   (wire (pts (xy 124.46 93.98) (xy 124.46 96.52))
     (stroke (width 0) (type default) (color 0 0 0 0))
@@
     (stroke (width 0) (type default) (color 0 0 0 0))
   )
-  (hierarchical_label "+5V" (shape input) (at 165.1 104.14 0)
+  (hierarchical_label "+5V" (shape input) (at 165.1 53.975 0)
     (effects (font (size 1.27 1.27)) (justify left))
   )
