File: Kc/MakerLAB_r03B/MakerLAB_r03B.kicad_pcb (KiCad board)
At the start: 2 copper layers, 374 x 178 mm, 153 parts, among them J1 Fix-Mod, J11 Conn_02x10_Counter_Clockwise, J12 Conn_02x05_Counter_Clockwise, J13 GND 0 1 2 3 4 5 6 7 +5V, J14 8Bit Jumper, J15 GND 0 1 2 3 4 5 6 7 +5V, J16 Conn_02x05_Counter_Clockwise, J17 Conn_02x10_Counter_Clockwise, J18 Conn_02x05_Counter_Clockwise, J19 Conn_01x10_Female, J21 Conn_01x03, J22 Conn_02x20_Counter_Clockwise, J23 Conn_02x20_Counter_Clockwise, J24 Conn_02x20_Counter_Clockwise, J25 IR Emitter & Sensor, J26 Conn_01x06_Female, J29 Conn_01x02_Male, J30 Conn_01x02_Male, J33 Visible Light Sensor, J34 Conn_01x05, J4 Barrel_Jack_MountingPin, J5 Conn_01x02_Male, J9 Conn_02x05_Counter_Clockwise, Q1 2N3904, Q2 2N3904, Q3 2N3904, Q4 2N3904, Q5 BC237, Q6 H21A1, SW1 SwGenerale, SW2 SW_DIP_x08, SW5 SW_Rotary12, U1 LM317_TO-220, U10 9368, U11 L78L33_SOT89, U12 HC-05 (ZC142200), U2 LM7805_TO220, U3 DM9368, U4 CC56-12EWA, U5 ULN2803A, U7 NE555P, U9 9368

Commit message: versione r03B della notte del 28 marzo 2023
Parts:
- removed J18: Conn_02x05_Counter_Clockwise, Connector_PinSocket_2.54mm:PinSocket_2x05_P2.54mm_Vertical
- added C11: 1uF, Capacitor_THT:C_Axial_L5.1mm_D3.1mm_P7.50mm_Horizontal, F.Cu at (151.5, 217.2)
- added C12: 1uF, Capacitor_THT:C_Axial_L5.1mm_D3.1mm_P7.50mm_Horizontal, F.Cu at (120.9, 217.2)
- added D15: LED, LED_THT:LED_D3.0mm, F.Cu at (118.9, 243.3)
- added D16: LED, LED_THT:LED_D3.0mm, F.Cu at (141.0, 243.3)
- added D18: LED, LED_THT:LED_D3.0mm, F.Cu at (181.4, 234.7)
- added D19: LED, LED_THT:LED_D3.0mm, F.Cu at (165.1, 234.7)
- added J2: Conn_02x05_Counter_Clockwise, Connector_PinSocket_2.54mm:PinSocket_2x05_P2.54mm_Vertical, F.Cu at (178.3, 244.6)
- added R10: 100, Resistor_THT:R_Axial_DIN0207_L6.3mm_D2.5mm_P10.16mm_Horizontal, F.Cu at (114.3, 226.1)
- added R11: 10K, Resistor_THT:R_Axial_DIN0207_L6.3mm_D2.5mm_P10.16mm_Horizontal, F.Cu at (138.8, 215.9)
- added R12: 10K, Resistor_THT:R_Axial_DIN0207_L6.3mm_D2.5mm_P10.16mm_Horizontal, F.Cu at (107.7, 226.1)
- added R13: 330, Resistor_THT:R_Axial_DIN0207_L6.3mm_D2.5mm_P10.16mm_Horizontal, F.Cu at (107.7, 231.1)
- added R14: 330, Resistor_THT:R_Axial_DIN0207_L6.3mm_D2.5mm_P10.16mm_Horizontal, F.Cu at (151.5, 231.1)
- added R18: 10K, Resistor_THT:R_Axial_DIN0207_L6.3mm_D2.5mm_P10.16mm_Horizontal, F.Cu at (163.1, 213.9)
- added R19: 10K, Resistor_THT:R_Axial_DIN0207_L6.3mm_D2.5mm_P10.16mm_Horizontal, F.Cu at (177.3, 213.9)
- added R20: 330, Resistor_THT:R_Axial_DIN0207_L6.3mm_D2.5mm_P10.16mm_Horizontal, F.Cu at (188.5, 230.1)
- added R21: 330, Resistor_THT:R_Axial_DIN0207_L6.3mm_D2.5mm_P10.16mm_Horizontal, F.Cu at (158.5, 240.3)
- added R9: 100, Resistor_THT:R_Axial_DIN0207_L6.3mm_D2.5mm_P10.16mm_Horizontal, F.Cu at (144.9, 226.0)
- added SW3: SW_Push, Button_Switch_THT:SW_Tactile_Straight_KSL0Axx1LFTR, F.Cu at (138.5, 231.6)
- added SW4: SW_Push, Button_Switch_THT:SW_Tactile_Straight_KSL0Axx1LFTR, F.Cu at (114.0, 231.1)
- added SW6: SW_Push, Button_Switch_THT:SW_Tactile_Straight_KSL0Axx1LFTR, F.Cu at (188.7, 226.6)
- added SW7: SW_Push, Button_Switch_THT:SW_Tactile_Straight_KSL0Axx1LFTR, F.Cu at (165.9, 226.6)
- added U6: 74LS14, Package_DIP:DIP-14_W7.62mm, F.Cu at (126.3, 216.2)
- added U8: 74LS00, Package_DIP:DIP-14_W7.62mm, F.Cu at (169.7, 218.9)
- moved J16 19.4 mm to (136.1, 244.6), turned to -90 degrees
Connections:
- C21 pad 1: Net-(C21-Pad1) -> /Alimentazione/+5V
- C22 pad 1: Net-(C21-Pad1) -> /Alimentazione/+5V
- J16 pad 1: /Pulse_2/Pulse+ -> GND
- J16 pad 10: /Pulse_2/Pulse+ -> /Pulse_2/Pulse-
- J16 pad 2: /Pulse_2/Pulse+ -> GND
- J16 pad 3: GND -> /Pulse_2/Pulse+
- J16 pad 4: /Pulse_2/Pulse- -> /Pulse_2/Pulse+
- J16 pad 5: /Pulse_2/Pulse- -> /Pulse_2/Pulse+
- J16 pad 6: /Pulse_2/Pulse- -> /Pulse_2/Pulse+
- J16 pad 8: GND -> /Pulse_2/Pulse-
- J16 pad 9: /Pulse_2/Pulse+ -> /Pulse_2/Pulse-
