File: Kc/MakerLAB_r03B/MakerLAB_r03B.kicad_sch (KiCad schematic)
At the start: 4 parts

Commit message: versione r03B della notte del 28 marzo 2023
Other:
- removed sheet Tastiera4x4
- sheet Gen_Clock ports: added none; removed Clock
- sheet Gen_fronti ports: added none; removed OUT+, OUT-
- sheet Pulse_2 ports: added none; removed Pulse+, Pulse-
