File: Kc/MakerLAB_r03B/Pulse_2.kicad_sch (KiCad schematic)
At the start: 14 parts, among them J16 Conn_02x05_Counter_Clockwise, SW3 SW_Push, SW4 SW_Push, U6 74LS14

Commit message: versione r03B della notte del 28 marzo 2023
Parts:
- C11, C12: footprint (none) -> Capacitor_THT:C_Axial_L5.1mm_D3.1mm_P7.50mm_Horizontal
- D15, D16: footprint (none) -> LED_THT:LED_D3.0mm
- R10, R11, R12, R13, R14, R9: footprint (none) -> Resistor_THT:R_Axial_DIN0207_L6.3mm_D2.5mm_P10.16mm_Horizontal
- SW3, SW4: footprint (none) -> Button_Switch_THT:SW_Tactile_Straight_KSL0Axx1LFTR
- U6: footprint (none) -> Package_DIP:DIP-14_W7.62mm
Connections:
- net VCC is gone; now on net +5V: R12.1
- net GND: now also J16.1 (Pin_1), J16.2 (Pin_2); no longer J16.3 (Pin_3), J16.8 (Pin_8)
- removed net Pulse+: J16.1 (Pin_1), J16.10 (Pin_10), J16.2 (Pin_2), J16.9 (Pin_9), U6.10
- net Pulse-: no longer names the net of J16.4 (Pin_4), J16.5 (Pin_5), J16.6 (Pin_6)
- net Pulse-: now also J16.3 (Pin_3), U6.10; no longer J16.7 (Pin_7), U6.4
- new net: J16.10 (Pin_10), J16.7 (Pin_7), J16.8 (Pin_8), J16.9 (Pin_9), U6.4
