File: Kc/MakerLAB_r03B/Visual2dgt.kicad_sch (KiCad schematic)
At the start: 12 parts, among them J19 Conn_01x10_Female, U10 9368, U9 9368

Commit message: versione r03B della notte del 28 marzo 2023
Connections:
- net +5V: now also C21.1, C22.1
Other:
- moved on the sheet: C21, C22
Changed lines of the file:
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@@
   (junction (at 182.88 63.5) (diameter 0) (color 0 0 0 0)
   )
+  (junction (at 135.89 52.07) (diameter 0) (color 0 0 0 0)
+  )
   (junction (at 83.82 33.02) (diameter 0) (color 0 0 0 0)
   )
@@
   (junction (at 182.88 88.9) (diameter 0) (color 0 0 0 0)
   )
-  (junction (at 80.01 99.06) (diameter 0) (color 0 0 0 0)
+  (junction (at 135.89 29.21) (diameter 0) (color 0 0 0 0)
+  )
+  (junction (at 135.89 59.69) (diameter 0) (color 0 0 0 0)
   )
   (junction (at 94.615 48.26) (diameter 0) (color 0 0 0 0)
@@
     (stroke (width 0) (type default) (color 0 0 0 0))
   )
-  (wire (pts (xy 80.01 99.06) (xy 86.36 99.06))
+  (wire (pts (xy 135.89 59.69) (xy 142.24 59.69))
     (stroke (width 0) (type default) (color 0 0 0 0))
   )
@@
     (stroke (width 0) (type default) (color 0 0 0 0))
   )
+  (wire (pts (xy 135.89 29.21) (xy 135.89 52.07))
+    (stroke (width 0) (type default) (color 0 0 0 0))
+  )
   (wire (pts (xy 189.23 73.66) (xy 186.69 73.66))
     (stroke (width 0) (type default) (color 0 0 0 0))
@@
     (stroke (width 0) (type default) (color 0 0 0 0))
   )
-  (wire (pts (xy 72.39 91.44) (xy 86.36 91.44))
+  (wire (pts (xy 128.27 52.07) (xy 135.89 52.07))
     (stroke (width 0) (type default) (color 0 0 0 0))
   )
@@
     (stroke (width 0) (type default) (color 0 0 0 0))
   )
+  (wire (pts (xy 135.89 52.07) (xy 142.24 52.07))
+    (stroke (width 0) (type default) (color 0 0 0 0))
+  )
   (wire (pts (xy 50.8 63.5) (xy 57.15 63.5))
     (stroke (width 0) (type default) (color 0 0 0 0))
@@
     (stroke (width 0) (type default) (color 0 0 0 0))
   )
-  (wire (pts (xy 72.39 99.06) (xy 80.01 99.06))
+  (wire (pts (xy 128.27 59.69) (xy 135.89 59.69))
     (stroke (width 0) (type default) (color 0 0 0 0))
   )
@@
     (stroke (width 0) (type default) (color 0 0 0 0))
   )
+  (wire (pts (xy 135.89 29.21) (xy 39.37 29.21))
+    (stroke (width 0) (type default) (color 0 0 0 0))
+  )
   (wire (pts (xy 208.28 91.44) (xy 226.06 91.44))
     (stroke (width 0) (type default) (color 0 0 0 0))
@@
     (stroke (width 0) (type default) (color 0 0 0 0))
   )
-  (wire (pts (xy 205.74 29.21) (xy 39.37 29.21))
+  (wire (pts (xy 205.74 29.21) (xy 135.89 29.21))
     (stroke (width 0) (type default) (color 0 0 0 0))
   )
@@
     (effects (font (size 1.27 1.27)) (justify right))
   )
-  (symbol (lib_id "Device:C") (at 72.39 95.25 0) (unit 1)
-    (in_bom yes) (on_board yes)
-    (property "Reference" "C21" (id 0) (at 75.565 93.98 0)
-      (effects (font (size 1.27 1.27)) (justify left))
-    )
-    (property "Value" "100n" (id 1) (at 75.565 96.52 0)
-      (effects (font (size 1.27 1.27)) (justify left))
-    )
-    (property "Footprint" "Capacitor_THT:C_Disc_D4.3mm_W1.9mm_P5.00mm" (id 2) (at 73.3552 99.06 0)
-      (effects (font (size 1.27 1.27)) hide)
-    )
-    (property "Datasheet" "~" (id 3) (at 72.39 95.25 0)
+  (symbol (lib_id "Device:C") (at 128.27 55.88 0) (unit 1)
+    (in_bom yes) (on_board yes)
+    (property "Reference" "C21" (id 0) (at 131.445 54.61 0)
+      (effects (font (size 1.27 1.27)) (justify left))
+    )
+    (property "Value" "100n" (id 1) (at 131.445 57.15 0)
+      (effects (font (size 1.27 1.27)) (justify left))
+    )
+    (property "Footprint" "Capacitor_THT:C_Disc_D4.3mm_W1.9mm_P5.00mm" (id 2) (at 129.2352 59.69 0)
+      (effects (font (size 1.27 1.27)) hide)
+    )
+    (property "Datasheet" "~" (id 3) (at 128.27 55.88 0)
       (effects (font (size 1.27 1.27)) hide)
     )
@@
     (pin "9")
   )
-  (symbol (lib_id "Device:C") (at 86.36 95.25 0) (unit 1)
-    (in_bom yes) (on_board yes)
-    (property "Reference" "C22" (id 0) (at 89.535 93.98 0)
-      (effects (font (size 1.27 1.27)) (justify left))
-    )
-    (property "Value" "100n" (id 1) (at 89.535 96.52 0)
-      (effects (font (size 1.27 1.27)) (justify left))
-    )
-    (property "Footprint" "Capacitor_THT:C_Disc_D4.3mm_W1.9mm_P5.00mm" (id 2) (at 87.3252 99.06 0)
-      (effects (font (size 1.27 1.27)) hide)
-    )
-    (property "Datasheet" "~" (id 3) (at 86.36 95.25 0)
+  (symbol (lib_id "Device:C") (at 142.24 55.88 0) (unit 1)
+    (in_bom yes) (on_board yes)
+    (property "Reference" "C22" (id 0) (at 145.415 54.61 0)
+      (effects (font (size 1.27 1.27)) (justify left))
+    )
+    (property "Value" "100n" (id 1) (at 145.415 57.15 0)
+      (effects (font (size 1.27 1.27)) (justify left))
+    )
+    (property "Footprint" "Capacitor_THT:C_Disc_D4.3mm_W1.9mm_P5.00mm" (id 2) (at 143.2052 59.69 0)
+      (effects (font (size 1.27 1.27)) hide)
+    )
+    (property "Datasheet" "~" (id 3) (at 142.24 55.88 0)
       (effects (font (size 1.27 1.27)) hide)
     )
@@
     (pin "3")
   )
-  (symbol (lib_id "power:GND") (at 80.01 99.06 0) (unit 1)
+  (symbol (lib_id "power:GND") (at 135.89 59.69 0) (unit 1)
     (in_bom yes) (on_board yes) (fields_autoplaced)
-    (property "Reference" "#PWR040" (id 0) (at 80.01 105.41 0)
-      (effects (font (size 1.27 1.27)) hide)
-    )
-    (property "Value" "GND" (id 1) (at 80.01 104.14 0))
-    (property "Footprint" "" (id 2) (at 80.01 99.06 0)
-      (effects (font (size 1.27 1.27)) hide)
-    )
-    (property "Datasheet" "" (id 3) (at 80.01 99.06 0)
-      (effects (font (size 1.27 1.27)) hide)
-    )
+    (property "Reference" "#PWR040" (id 0) (at 135.89 66.04 0)
+      (effects (font (size 1.27 1.27)) hide)
+    )
+    (property "Value" "GND" (id 1) (at 135.89 64.77 0))
+    (property "Footprint" "" (id 2) (at 135.89 59.69 0)
+      (effects (font (size 1.27 1.27)) hide)
+    )
+    (property "Datasheet" "" (id 3) (at 135.89 59.69 0)
+      (effects (font (size 1.27 1.27)) hide)
+    )
