File: Kc/MakerLAB_r011M/MakerLAB_r011M.kicad_pcb (KiCad board)
At the start: 2 copper layers, 374 x 178 mm, 173 parts, among them J1 Fix-Mod, J11 Conn_02x10_Counter_Clockwise, J12 Conn_02x05_Counter_Clockwise, J13 GND 0 1 2 3 4 5 6 7 +5V, J14 8Bit Jumper, J15 GND 0 1 2 3 4 5 6 7 +5V, J16 Conn_02x05_Counter_Clockwise, J17 Conn_02x10_Counter_Clockwise, J19 Conn_01x10_Female, J2 Conn_02x05_Counter_Clockwise, J21 Conn_01x03, J22 Conn_02x20_Counter_Clockwise, J23 Conn_02x20_Counter_Clockwise, J24 Conn_02x20_Counter_Clockwise, J25 IR Emitter & Sensor, J26 Conn_01x06_Female, J29 Conn_01x02_Male, J30 Conn_01x02_Male, J33 Visible Light Sensor, J34 Conn_01x05, J4 Barrel_Jack_MountingPin, J5 Conn_01x02_Male, J9 Conn_02x05_Counter_Clockwise, Q1 2N3904, Q2 2N3904, Q3 2N3904, Q4 2N3904, Q5 BC237, Q6 H21A1, Q7 BS170, Q8 BS170, SW1 SwGenerale, SW2 SW_DIP_x08, SW3 SW_Push, SW4 SW_Push, SW5 SW_Rotary12, SW6 SW_Push, SW7 SW_Push, U1 LM317_TO-220, U10 9368, U11 L78L33_SOT89, U12 HC-05 (ZC142200), U2 LM7805_TO220, U3 DM9368, U4 CC56-12EWA, U5 ULN2803A, U6 74LS14, U7 NE555P, U8 74LS00, U9 9368

Commit message: r03C
Parts:
- removed Q7, Q8: BS170, Package_TO_SOT_THT:TO-92_Inline
- removed R34, R35: 10K, Resistor_THT:R_Axial_DIN0207_L6.3mm_D2.5mm_P10.16mm_Horizontal
- added D23: 1n4148, Diode_THT:D_A-405_P10.16mm_Horizontal, F.Cu at (248.1, 99.6)
- added D24: 1n4148, Diode_THT:D_A-405_P10.16mm_Horizontal, F.Cu at (247.9, 104.7)
- added D25: 1n4148, Diode_THT:D_A-405_P10.16mm_Horizontal, F.Cu at (248.1, 80.0)
- added D26: 1n4148, Diode_THT:D_A-405_P10.16mm_Horizontal, F.Cu at (248.2, 75.1)
- added D27: 1n4148, Diode_THT:D_A-405_P10.16mm_Horizontal, F.Cu at (248.2, 70.2)
- added D6: 1n4148, Diode_THT:D_A-405_P10.16mm_Horizontal, F.Cu at (248.2, 94.6)
- R32, R33: value 10K -> 1K
- moved J16 119.5 mm to (136.1, 244.6), turned to -90 degrees
- moved J2 119.3 mm to (178.3, 244.6), turned to -90 degrees
- moved R13 116.3 mm to (107.7, 231.1)
- moved R12 112.7 mm to (107.7, 226.1)
- moved R21 110.4 mm to (158.5, 240.3)
- moved D16 110.4 mm to (141.0, 243.3), turned to 0 degrees
- moved R11 109.0 mm to (138.8, 215.9)
- moved R10 108.8 mm to (114.3, 226.1)
- moved D15 108.3 mm to (118.9, 243.3), turned to 180 degrees
- moved R19 103.9 mm to (177.3, 213.9), turned to 0 degrees
- moved D18 103.7 mm to (181.4, 234.7), turned to 0 degrees
- moved U8 101.1 mm to (169.7, 218.9)
- moved R20 100.6 mm to (188.5, 230.1)
- moved R9 100.4 mm to (144.9, 226.0)
- moved SW4 100.2 mm to (114.0, 231.1)
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Connections:
- net Net-(D17-Pad1) renamed /Gen_Clock/Clock
- net Net-(J16-Pad10) renamed /Pulse_2/Pulse-
- net Net-(J16-Pad3) renamed /Pulse_2/Pulse+
- net Net-(J2-Pad10) renamed /Gen_fronti/OUT-
- net Net-(J2-Pad3) renamed /Gen_fronti/OUT+
- R32 pad 2: /BT to Serial/+3.3V -> Net-(J34-Pad2)
- R33 pad 2: /BT to Serial/+3.3V -> Net-(J34-Pad3)
