File: Kc/MakerLAB_r03C/PadSerigrafie.kicad_sch (KiCad schematic)
At the start: 16 parts

Commit message: Routing e Zone OK
Parts:
- added TP31, TP32, TP34, TP35: Pulse Generator, SerigrafieMakerLab:Disp4x7Seg, symbol Connector:TestPoint
Other:
- moved on the sheet: TP28
Changed lines of the file:
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@@
+    (pin "1")
+  )
+  (symbol (lib_id "Connector:TestPoint") (at 124.46 132.08 0) (unit 1)
+    (in_bom yes) (on_board yes) (fields_autoplaced)
+    (property "Reference" "TP35" (id 0) (at 127 127.5079 0)
+      (effects (font (size 1.27 1.27)) (justify left))
+    )
+    (property "Value" "Pulse Generator" (id 1) (at 127 130.0479 0)
+      (effects (font (size 1.27 1.27)) (justify left))
+    )
+    (property "Footprint" "SerigrafieMakerLab:Disp4x7Seg" (id 2) (at 129.54 132.08 0)
+      (effects (font (size 1.27 1.27)) hide)
+    )
+    (property "Datasheet" "~" (id 3) (at 129.54 132.08 0)
+      (effects (font (size 1.27 1.27)) hide)
+    )
+    (pin "1")
+  )
+  (symbol (lib_id "Connector:TestPoint") (at 105.41 132.08 0) (unit 1)
+    (in_bom yes) (on_board yes) (fields_autoplaced)
+    (property "Reference" "TP34" (id 0) (at 107.95 127.5079 0)
+      (effects (font (size 1.27 1.27)) (justify left))
+    )
+    (property "Value" "Pulse Generator" (id 1) (at 107.95 130.0479 0)
+      (effects (font (size 1.27 1.27)) (justify left))
+    )
+    (property "Footprint" "SerigrafieMakerLab:Disp4x7Seg" (id 2) (at 110.49 132.08 0)
+      (effects (font (size 1.27 1.27)) hide)
+    )
+    (property "Datasheet" "~" (id 3) (at 110.49 132.08 0)
+      (effects (font (size 1.27 1.27)) hide)
+    )
     (pin "1")
   )
@@
     )
     (property "Datasheet" "~" (id 3) (at 44.45 60.96 0)
+      (effects (font (size 1.27 1.27)) hide)
+    )
+    (pin "1")
+  )
+  (symbol (lib_id "Connector:TestPoint") (at 87.63 132.08 0) (unit 1)
+    (in_bom yes) (on_board yes) (fields_autoplaced)
+    (property "Reference" "TP32" (id 0) (at 90.17 127.5079 0)
+      (effects (font (size 1.27 1.27)) (justify left))
+    )
+    (property "Value" "Pulse Generator" (id 1) (at 90.17 130.0479 0)
+      (effects (font (size 1.27 1.27)) (justify left))
+    )
+    (property "Footprint" "SerigrafieMakerLab:Disp4x7Seg" (id 2) (at 92.71 132.08 0)
+      (effects (font (size 1.27 1.27)) hide)
+    )
+    (property "Datasheet" "~" (id 3) (at 92.71 132.08 0)
       (effects (font (size 1.27 1.27)) hide)
     )
@@
     (pin "1")
   )
-  (symbol (lib_id "Connector:TestPoint") (at 87.63 129.54 0) (unit 1)
+  (symbol (lib_id "Connector:TestPoint") (at 87.63 158.75 0) (unit 1)
     (in_bom yes) (on_board yes) (fields_autoplaced)
-    (property "Reference" "TP28" (id 0) (at 90.17 123.6979 0)
+    (property "Reference" "TP28" (id 0) (at 90.17 152.9079 0)
       (effects (font (size 1.27 1.27)) (justify left))
     )
-    (property "Value" "MakerLAB" (id 1) (at 90.17 126.2379 0)
+    (property "Value" "MakerLAB" (id 1) (at 90.17 155.4479 0)
       (effects (font (size 1.27 1.27)) (justify left))
     )
-    (property "Footprint" "SerigrafieMakerLAB:MakerLABTitoli" (id 2) (at 90.17 128.7779 0)
+    (property "Footprint" "SerigrafieMakerLAB:MakerLABTitoli" (id 2) (at 90.17 157.9879 0)
       (effects (font (size 1.27 1.27)) (justify left))
     )
-    (property "Datasheet" "~" (id 3) (at 92.71 129.54 0)
+    (property "Datasheet" "~" (id 3) (at 92.71 158.75 0)
       (effects (font (size 1.27 1.27)) hide)
     )
@@
       (effects (font (size 1.27 1.27)) hide)
     )
+    (pin "1")
+  )
+  (symbol (lib_id "Connector:TestPoint") (at 71.12 132.08 0) (unit 1)
+    (in_bom yes) (on_board yes) (fields_autoplaced)
+    (property "Reference" "TP31" (id 0) (at 73.66 127.5079 0)
+      (effects (font (size 1.27 1.27)) (justify left))
+    )
+    (property "Value" "Pulse Generator" (id 1) (at 73.66 130.0479 0)
+      (effects (font (size 1.27 1.27)) (justify left))
+    )
+    (property "Footprint" "SerigrafieMakerLab:Disp4x7Seg" (id 2) (at 76.2 132.08 0)
+      (effects (font (size 1.27 1.27)) hide)
+    )
+    (property "Datasheet" "~" (id 3) (at 76.2 132.08 0)
+      (effects (font (size 1.27 1.27)) hide)
+    )
