File: Kc/MakerLAB_r03C/Visual_4Dgt.kicad_sch (KiCad schematic)
At the start: 15 parts, among them J11 Conn_02x10_Counter_Clockwise, J12 Conn_02x05_Counter_Clockwise, J9 Conn_02x05_Counter_Clockwise, Q1 2N3904, Q2 2N3904, Q3 2N3904, Q4 2N3904, U3 DM9368, U4 CC56-12EWA

Commit message: 20230404 2:20
Other:
- moved on the sheet: C8
Changed lines of the file:
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@@
   (junction (at 69.85 64.77) (diameter 0) (color 0 0 0 0)
+  )
+  (junction (at 59.69 20.32) (diameter 0) (color 0 0 0 0)
   )
   (junction (at 59.69 64.77) (diameter 0) (color 0 0 0 0)
@@
     (stroke (width 0) (type default) (color 0 0 0 0))
   )
-  (wire (pts (xy 59.69 21.59) (xy 59.69 31.75))
+  (wire (pts (xy 59.69 20.32) (xy 59.69 31.75))
     (stroke (width 0) (type default) (color 0 0 0 0))
   )
@@
     (stroke (width 0) (type default) (color 0 0 0 0))
   )
-  (wire (pts (xy 48.26 68.58) (xy 50.8 68.58))
-    (stroke (width 0) (type default) (color 0 0 0 0))
-  )
-  (wire (pts (xy 73.66 148.59) (xy 73.66 152.4))
+  (wire (pts (xy 59.69 20.32) (xy 61.595 20.32))
+    (stroke (width 0) (type default) (color 0 0 0 0))
+  )
+  (wire (pts (xy 19.05 20.32) (xy 19.05 24.13))
     (stroke (width 0) (type default) (color 0 0 0 0))
   )
@@
     (stroke (width 0) (type default) (color 0 0 0 0))
   )
+  (wire (pts (xy 19.05 20.32) (xy 59.69 20.32))
+    (stroke (width 0) (type default) (color 0 0 0 0))
+  )
   (wire (pts (xy 185.42 80.01) (xy 178.435 80.01))
     (stroke (width 0) (type default) (color 0 0 0 0))
@@
     (stroke (width 0) (type default) (color 0 0 0 0))
   )
-  (wire (pts (xy 73.66 160.02) (xy 73.66 163.83))
+  (wire (pts (xy 19.05 31.75) (xy 19.05 35.56))
     (stroke (width 0) (type default) (color 0 0 0 0))
   )
@@
     (stroke (width 0) (type default) (color 0 0 0 0))
   )
-  (wire (pts (xy 50.8 64.77) (xy 59.69 64.77))
-    (stroke (width 0) (type default) (color 0 0 0 0))
-  )
   (wire (pts (xy 195.58 99.06) (xy 270.51 99.06))
     (stroke (width 0) (type default) (color 0 0 0 0))
@@
   )
   (wire (pts (xy 262.89 111.76) (xy 256.54 111.76))
-    (stroke (width 0) (type default) (color 0 0 0 0))
-  )
-  (wire (pts (xy 50.8 64.77) (xy 50.8 68.58))
     (stroke (width 0) (type default) (color 0 0 0 0))
   )
@@
     (effects (font (size 1.27 1.27)) (justify left bottom))
   )
-  (hierarchical_label "GND_pwr" (shape input) (at 48.26 68.58 180)
-    (effects (font (size 1.27 1.27)) (justify right))
-  )
-  (symbol (lib_id "power:+5V") (at 59.69 21.59 0) (unit 1)
-    (in_bom yes) (on_board yes)
-    (property "Reference" "#PWR06" (id 0) (at 59.69 25.4 0)
-      (effects (font (size 1.27 1.27)) hide)
-    )
-    (property "Value" "+5V" (id 1) (at 60.071 17.1958 0))
-    (property "Footprint" "" (id 2) (at 59.69 21.59 0)
-      (effects (font (size 1.27 1.27)) hide)
-    )
-    (property "Datasheet" "" (id 3) (at 59.69 21.59 0)
-      (effects (font (size 1.27 1.27)) hide)
-    )
-    (pin "1")
+  (hierarchical_label "+5V" (shape input) (at 61.595 20.32 0)
+    (effects (font (size 1.27 1.27)) (justify left))
   )
   (symbol (lib_id "power:GND") (at 119.38 119.38 0) (unit 1)
@@
     (pin "1")
     (pin "2")
-  )
-  (symbol (lib_id "power:+5V") (at 73.66 148.59 0) (unit 1)
-    (in_bom yes) (on_board yes)
-    (property "Reference" "#PWR08" (id 0) (at 73.66 152.4 0)
-      (effects (font (size 1.27 1.27)) hide)
-    )
-    (property "Value" "+5V" (id 1) (at 74.041 144.1958 0))
-    (property "Footprint" "" (id 2) (at 73.66 148.59 0)
-      (effects (font (size 1.27 1.27)) hide)
-    )
-    (property "Datasheet" "" (id 3) (at 73.66 148.59 0)
-      (effects (font (size 1.27 1.27)) hide)
-    )
-    (pin "1")
   )
   (symbol (lib_id "Connector_Generic:Conn_02x05_Odd_Even") (at 190.5 85.09 90) (mirror x) (unit 1)
@@
     (pin "9")
   )
-  (symbol (lib_id "power:GND") (at 73.66 163.83 0) (unit 1)
-    (in_bom yes) (on_board yes)
-    (property "Reference" "#PWR09" (id 0) (at 73.66 170.18 0)
-      (effects (font (size 1.27 1.27)) hide)
-    )
-    (property "Value" "GND" (id 1) (at 73.787 168.2242 0))
-    (property "Footprint" "" (id 2) (at 73.66 163.83 0)
-      (effects (font (size 1.27 1.27)) hide)
-    )
-    (property "Datasheet" "" (id 3) (at 73.66 163.83 0)
+  (symbol (lib_id "power:GND") (at 19.05 35.56 0) (unit 1)
+    (in_bom yes) (on_board yes)
+    (property "Reference" "#PWR09" (id 0) (at 19.05 41.91 0)
+      (effects (font (size 1.27 1.27)) hide)
+    )
+    (property "Value" "GND" (id 1) (at 19.177 39.9542 0))
+    (property "Footprint" "" (id 2) (at 19.05 35.56 0)
+      (effects (font (size 1.27 1.27)) hide)
+    )
+    (property "Datasheet" "" (id 3) (at 19.05 35.56 0)
       (effects (font (size 1.27 1.27)) hide)
     )
@@
     (pin "1")
   )
-  (symbol (lib_id "Device:C") (at 73.66 156.21 0) (unit 1)
-    (in_bom yes) (on_board yes)
-    (property "Reference" "C8" (id 0) (at 76.581 155.0416 0)
+  (symbol (lib_id "Device:C") (at 19.05 27.94 0) (unit 1)
+    (in_bom yes) (on_board yes)
+    (property "Reference" "C8" (id 0) (at 21.971 26.7716 0)
       (effects (font (size 1.27 1.27)) (justify left))
     )
-    (property "Value" "100nF" (id 1) (at 76.581 157.353 0)
+    (property "Value" "100nF" (id 1) (at 21.971 29.083 0)
       (effects (font (size 1.27 1.27)) (justify left))
     )
-    (property "Footprint" "Capacitor_THT:C_Disc_D7.5mm_W2.5mm_P5.00mm" (id 2) (at 74.6252 160.02 0)
-      (effects (font (size 1.27 1.27)) hide)
-    )
-    (property "Datasheet" "~" (id 3) (at 73.66 156.21 0)
-      (effects (font (size 1.27 1.27)) hide)
-    )
+    (property "Footprint" "Capacitor_THT:C_Disc_D7.5mm_W2.5mm_P5.00mm" (id 2) (at 20.0152 31.75 0)
+      (effects (font (size 1.27 1.27)) hide)
+    )
+    (property "Datasheet" "~" (id 3) (at 19.05 27.94 0)
+      (effects (font (size 1.27 1.27)) hide)
+    )

Commit message: 20230404 14:30
Connections:
- net GND: now also J11.1 (Pin_1), J11.2 (Pin_2), J11.3 (Pin_3), J11.4 (Pin_4), J11.6 (Pin_6); no longer J11.15 (Pin_15), J11.17 (Pin_17)
- net at U4.1 (e): now also J11.15 (Pin_15); no longer J11.10 (Pin_10)
- net at U4.10 (f): now also J11.17 (Pin_17); no longer J11.12 (Pin_12)
- net at U4.11 (a): now also J11.7 (Pin_7); no longer J11.2 (Pin_2)
- net at U4.2 (d): now also J11.13 (Pin_13); no longer J11.8 (Pin_8)
- net at R4.2, U4.3 (DPX): no longer J11.16 (Pin_16)
- net at U4.4 (c): now also J11.11 (Pin_11); no longer J11.6 (Pin_6)
- net at U4.5 (g): now also J11.19 (Pin_19); no longer J11.14 (Pin_14)
- net at U4.7 (b): now also J11.9 (Pin_9); no longer J11.4 (Pin_4)
- net at U3.13 (a): now also J11.8 (Pin_8); no longer J11.1 (Pin_1)
- net at U3.15 (f): now also J11.18 (Pin_18); no longer J11.11 (Pin_11)
- net at U3.14 (g): now also J11.20 (Pin_20); no longer J11.13 (Pin_13)
- net at R4.1: now also J11.5 (Pin_5); no longer J11.20 (Pin_20)
- net at U3.12 (b): now also J11.10 (Pin_10); no longer J11.3 (Pin_3)
- net at U3.11 (c): now also J11.12 (Pin_12); no longer J11.5 (Pin_5)
- net at U3.10 (d): now also J11.14 (Pin_14); no longer J11.7 (Pin_7)
- net at U3.9 (e): now also J11.16 (Pin_16); no longer J11.9 (Pin_9)
- no-connect marks 3 -> 2
Other:
- moved on the sheet: J11, R4, U4

Commit message: Routing e Zone OK
Parts:
- J11: value Conn_02x10_Counter_Clockwise -> 1 2 3 4 5
Changed lines of the file:
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@@
   )
   (symbol (lib_id "Connector_Generic:Conn_02x10_Odd_Even") (at 80.01 41.91 0) (mirror y) (unit 1)
-    (in_bom yes) (on_board yes) (fields_autoplaced)
+    (in_bom yes) (on_board yes)
     (property "Reference" "J11" (id 0) (at 78.74 25.4 0))
-    (property "Value" "Conn_02x10_Counter_Clockwise" (id 1) (at 78.74 27.94 0))
+    (property "Value" "1 2 3 4 5" (id 1) (at 78.74 27.94 0))
     (property "Footprint" "Connector_PinSocket_2.54mm:PinSocket_2x10_P2.54mm_Vertical" (id 2) (at 80.01 41.91 0)
       (effects (font (size 1.27 1.27)) hide)

Commit message: test schematic scritte
Parts:
- J11: value 1 2 3 4 5 -> g f e d c b a
Changed lines of the file:
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@@
     (in_bom yes) (on_board yes)
     (property "Reference" "J11" (id 0) (at 78.74 25.4 0))
-    (property "Value" "1 2 3 4 5" (id 1) (at 78.74 27.94 0))
+    (property "Value" "g  f  e  d c  b  a" (id 1) (at 88.9 46.99 90))
     (property "Footprint" "Connector_PinSocket_2.54mm:PinSocket_2x10_P2.54mm_Vertical" (id 2) (at 80.01 41.91 0)
       (effects (font (size 1.27 1.27)) hide)

Commit message: visual 4 dgt scritte
Parts:
- J11: value g f e d c b a -> Gnd Dp a b c d e f g
- J9: value Conn_02x05_Counter_Clockwise -> D C B A LE
Changed lines of the file:
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@@
   )
   (symbol (lib_id "Connector_Generic:Conn_02x05_Odd_Even") (at 24.13 86.36 90) (unit 1)
-    (in_bom yes) (on_board yes) (fields_autoplaced)
+    (in_bom yes) (on_board yes)
     (property "Reference" "J9" (id 0) (at 31.75 83.8199 90)
       (effects (font (size 1.27 1.27)) (justify right))
     )
-    (property "Value" "Conn_02x05_Counter_Clockwise" (id 1) (at 31.75 86.3599 90)
+    (property "Value" "D C B A  LE" (id 1) (at 19.05 78.74 90)
       (effects (font (size 1.27 1.27)) (justify right))
     )
@@
     (in_bom yes) (on_board yes)
     (property "Reference" "J11" (id 0) (at 78.74 25.4 0))
-    (property "Value" "g  f  e  d c  b  a" (id 1) (at 88.9 46.99 90))
+    (property "Value" "Gnd Dp a  b  c  d e  f  g  " (id 1) (at 88.9 46.99 90))
     (property "Footprint" "Connector_PinSocket_2.54mm:PinSocket_2x10_P2.54mm_Vertical" (id 2) (at 80.01 41.91 0)
       (effects (font (size 1.27 1.27)) hide)

Commit message: 4 DGT SCRITTE 2
Parts:
- J11: value Gnd Dp a b c d e f g -> Gnd Dp a b c d e f g
Changed lines of the file:
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@@
     (in_bom yes) (on_board yes)
     (property "Reference" "J11" (id 0) (at 78.74 25.4 0))
-    (property "Value" "Gnd Dp a  b  c  d e  f  g  " (id 1) (at 88.9 46.99 90))
+    (property "Value" "Gnd Dp a  b  c  d   e   f   g  " (id 1) (at 80.01 60.96 0))
     (property "Footprint" "Connector_PinSocket_2.54mm:PinSocket_2x10_P2.54mm_Vertical" (id 2) (at 80.01 41.91 0)
       (effects (font (size 1.27 1.27)) hide)
