File: Kc/MakerLAB_r03C/MakerLAB_r03C.kicad_pcb (KiCad board)
At the start: 2 copper layers, 374 x 178 mm, 173 parts, among them J1 Fix-Mod, J11 Conn_02x10_Counter_Clockwise, J12 Conn_02x05_Counter_Clockwise, J13 GND 0 1 2 3 4 5 6 7 +5V, J14 8Bit Jumper, J15 GND 0 1 2 3 4 5 6 7 +5V, J16 Conn_02x05_Counter_Clockwise, J17 Conn_02x10_Counter_Clockwise, J19 Conn_01x10_Female, J2 Conn_02x05_Counter_Clockwise, J21 Conn_01x03, J22 Conn_02x20_Counter_Clockwise, J23 Conn_02x20_Counter_Clockwise, J24 Conn_02x20_Counter_Clockwise, J25 IR Emitter & Sensor, J26 Conn_01x06_Female, J29 Conn_01x02_Male, J30 Conn_01x02_Male, J33 Visible Light Sensor, J34 Conn_01x05, J4 Barrel_Jack_MountingPin, J5 Conn_01x02_Male, J9 Conn_02x05_Counter_Clockwise, Q1 2N3904, Q2 2N3904, Q3 2N3904, Q4 2N3904, Q5 BC237, Q6 H21A1, Q7 BS170, Q8 BS170, SW1 SwGenerale, SW2 SW_DIP_x08, SW3 SW_Push, SW4 SW_Push, SW5 SW_Rotary12, SW6 SW_Push, SW7 SW_Push, U1 LM317_TO-220, U10 9368, U11 L78L33_SOT89, U12 HC-05 (ZC142200), U2 LM7805_TO220, U3 DM9368, U4 CC56-12EWA, U5 ULN2803A, U6 74LS14, U7 NE555P, U8 74LS00, U9 9368

Commit message: r03C
Parts:
- removed TP30: Pulse Generator, SerigrafieMakerLAB:Clock NE555
- added +5: Conn_01x05, Connector_PinHeader_2.54mm:PinHeader_1x05_P2.54mm_Vertical, F.Cu at (264.7, 36.9)
- added +Var1: Conn_01x05, Connector_PinHeader_2.54mm:PinHeader_1x05_P2.54mm_Vertical, F.Cu at (255.5, 36.9)
- added C13: 100nF, Capacitor_THT:C_Axial_L5.1mm_D3.1mm_P7.50mm_Horizontal, F.Cu at (119.5, 134.6)
- added C15: 10nF, Capacitor_THT:C_Axial_L5.1mm_D3.1mm_P7.50mm_Horizontal, F.Cu at (119.5, 145.2)
- added GND1: Conn_01x05, Connector_PinHeader_2.54mm:PinHeader_1x05_P2.54mm_Vertical, F.Cu at (250.9, 36.9)
- added R4: 330, Resistor_THT:R_Axial_DIN0207_L6.3mm_D2.5mm_P10.16mm_Horizontal, F.Cu at (122.8, 39.8)
- added TP29: 8 x LED, SerigrafieMakerLab:Clock NE555, F.Cu at (98.7, 133.2)
- moved +3.3 14.9 mm to (260.1, 36.9)
Connections:
- TP1 pad 1: GNDA -> GND
- TP2 pad 1: GNDA -> GND
- TP20 pad 1: GNDA -> GND
- TP3 pad 1: GNDA -> GND
- TP4 pad 1: GNDA -> GND
- TP5 pad 1: GNDA -> GND
Routing:
- net Net-(C16-Pad1): track 175.5 -> 0.00 mm
- net Net-(C1-Pad1): track 172.6 -> 0.00 mm
- net /Alimentazione/+Vvar: track 95.3 -> 0.00 mm
- net Net-(C24-Pad1): track 84.6 -> 0.00 mm
- net Net-(C4-Pad1): track 69.6 -> 0.00 mm
- net Net-(C7-Pad1): track 63.3 -> 0.00 mm
- net Net-(J4-Pad2): track 38.3 -> 0.00 mm
- net Net-(D1-Pad1): track 37.5 -> 0.00 mm
- net Net-(D2-Pad1): track 23.6 -> 0.00 mm
- net Net-(D1-Pad2): track 22.8 -> 0.00 mm
- net /Alimentazione/+3.3V: track 16.2 -> 0.00 mm
- net /Alimentazione/+5V: track 16.1 -> 0.00 mm
- net Net-(F1-Pad1): track 12.8 -> 0.00 mm
- net Net-(D22-Pad2): track 12.1 -> 0.00 mm
- net Net-(D21-Pad2): track 10.8 -> 0.00 mm
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- removed copper zone on B.Cu, net GND
- removed copper zone on F.Cu, net GND

Commit message: 20230403 - Routing in corso
Routing:
- net GND: track 0.00 -> 1701.1 mm, vias 0 -> 1
- net /Alimentazione/+5V: track 0.00 -> 986.5 mm, vias 0 -> 1
- net /Alimentazione/+Vvar: track 0.00 -> 379.6 mm
- net /Alimentazione/+3.3V: track 0.00 -> 309.0 mm
- net Net-(C16-Pad1): track 0.00 -> 177.8 mm
- net Net-(C1-Pad1): track 0.00 -> 158.1 mm
- net Net-(D17-Pad1): track 0.00 -> 125.4 mm, vias 0 -> 1
- net Net-(C4-Pad1): track 0.00 -> 92.3 mm
- net Net-(C24-Pad1): track 0.00 -> 85.4 mm
- net Net-(J19-Pad8): track 0.00 -> 84.3 mm, vias 0 -> 2
- net Net-(J9-Pad9): track 0.00 -> 70.1 mm
- net Net-(J26-Pad4): track 0.00 -> 69.8 mm
- net Net-(J2-Pad10): track 0.00 -> 69.2 mm
- net Net-(J19-Pad5): track 0.00 -> 68.3 mm
- net Net-(J9-Pad10): track 0.00 -> 66.2 mm
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
Commit message: 20230403 17:12
Routing:
- net /Alimentazione/+5V: track 986.5 -> 1188.8 mm, vias 1 -> 0
- net /Alimentazione/+3.3V: track 309.0 -> 348.0 mm
- net Net-(J19-Pad1): track 57.5 -> 61.6 mm
- net /Alimentazione/+Vvar: track 379.6 -> 376.4 mm

Commit message: 20230404 2:20
Parts:
- moved D20 16.5 mm to (26.7, 90.9)
Connections:
- C8 pad 1: +5V -> /Alimentazione/+5V
- U3 pad 16: +5V -> /Alimentazione/+5V
- U7 pad 4: unconnected-(U7-Pad4) -> /Alimentazione/+5V
Routing:
- net GND: track 1701.1 -> 591.0 mm, vias 1 -> 130
- net /Alimentazione/+5V: track 1188.8 -> 1531.1 mm, vias 0 -> 17
- net Net-(C16-Pad1): track 177.8 -> 218.4 mm
- net +5V: track 27.8 -> 0.00 mm
- net Net-(C1-Pad1): track 158.1 -> 177.4 mm
- net Net-(J2-Pad10): track 69.2 -> 55.4 mm
- net Net-(J9-Pad10): track 66.2 -> 55.1 mm
- net Net-(AFF2-Pad4): track 10.1 -> 17.9 mm
- net /Alimentazione/+Vvar: track 376.4 -> 384.2 mm
- net /Alimentazione/+3.3V: track 348.0 -> 355.6 mm
- net Net-(RV3-Pad2): track 65.7 -> 58.6 mm
- net Net-(AFF2-Pad10): track 53.3 -> 58.6 mm
- net Net-(C7-Pad1): track 55.9 -> 60.7 mm
- net Net-(J26-Pad4): track 69.8 -> 65.1 mm
- net Net-(U10-Pad2): track 22.5 -> 18.2 mm
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- added copper zone on B.Cu, net GND
- added copper zone on F.Cu, net GND

Commit message: 20230404 14:30
Parts:
- removed J17: Conn_02x10_Counter_Clockwise, Connector_PinHeader_2.54mm:PinHeader_2x10_P2.54mm_Vertical
- added J3: Conn_02x10_Counter_Clockwise, Connector_PinSocket_2.54mm:PinSocket_2x10_P2.54mm_Vertical, F.Cu at (173.9, 135.0)
- moved R4 20.9 mm to (143.7, 38.7), turned to 180 degrees
- moved C3 10.9 mm to (22.3, 127.6)
- moved Q1 2.21 mm to (118.6, 44.4)
- moved Q2 2.21 mm to (125.0, 44.5)
- moved Q3 2.21 mm to (131.3, 44.5)
- moved Q4 2.21 mm to (137.3, 44.6)
- moved LCD1 0.65 mm to (143.7, 86.5)
Connections:
- J11 pad 1: Net-(J11-Pad1) -> GND
- J11 pad 15: GND -> Net-(J11-Pad15)
- J11 pad 17: GND -> Net-(J11-Pad17)
- J11 pad 18: unconnected-(J11-Pad18) -> Net-(J11-Pad18)
- J11 pad 19: unconnected-(J11-Pad19) -> Net-(J11-Pad19)
- J11 pad 2: Net-(J11-Pad2) -> GND
- J11 pad 3: Net-(J11-Pad3) -> GND
- J11 pad 4: Net-(J11-Pad4) -> GND
- J11 pad 6: Net-(J11-Pad6) -> GND
- R4 pad 1: Net-(J11-Pad20) -> Net-(J11-Pad5)
- R4 pad 2: Net-(J11-Pad16) -> Net-(R4-Pad2)
- U3 pad 10: Net-(J11-Pad7) -> Net-(J11-Pad14)
- U3 pad 11: Net-(J11-Pad5) -> Net-(J11-Pad12)
- U3 pad 12: Net-(J11-Pad3) -> Net-(J11-Pad10)
- U3 pad 13: Net-(J11-Pad1) -> Net-(J11-Pad8)
- U3 pad 14: Net-(J11-Pad13) -> Net-(J11-Pad20)
- U3 pad 15: Net-(J11-Pad11) -> Net-(J11-Pad18)
- U3 pad 9: Net-(J11-Pad9) -> Net-(J11-Pad16)
- U4 pad 1: Net-(J11-Pad10) -> Net-(J11-Pad15)
- U4 pad 10: Net-(J11-Pad12) -> Net-(J11-Pad17)
- U4 pad 11: Net-(J11-Pad2) -> Net-(J11-Pad7)
- U4 pad 2: Net-(J11-Pad8) -> Net-(J11-Pad13)
- U4 pad 3: Net-(J11-Pad16) -> Net-(R4-Pad2)
- U4 pad 4: Net-(J11-Pad6) -> Net-(J11-Pad11)
- U4 pad 5: Net-(J11-Pad14) -> Net-(J11-Pad19)
- U4 pad 7: Net-(J11-Pad4) -> Net-(J11-Pad9)
Routing:
- net GND: track 591.0 -> 286.9 mm, vias 130 -> 128
- net Net-(C16-Pad1): track 218.4 -> 290.0 mm
- net Net-(J11-Pad2): track 41.7 -> 0.00 mm, vias 1 -> 0
- net Net-(J11-Pad15): track 0.00 -> 37.5 mm
- net Net-(J11-Pad17): track 0.00 -> 37.2 mm
- net Net-(J11-Pad4): track 35.4 -> 0.00 mm
- net Net-(J11-Pad1): track 31.0 -> 0.00 mm, vias 1 -> 0
- net Net-(J11-Pad12): track 48.6 -> 17.7 mm, vias 1 -> 0
- net Net-(J11-Pad18): track 0.00 -> 29.9 mm, vias 0 -> 1
- net Net-(J11-Pad3): track 28.5 -> 0.00 mm, vias 1 -> 0
- net Net-(D1-Pad1): track 50.2 -> 22.6 mm
- net Net-(J11-Pad16): track 44.0 -> 17.7 mm, vias 1 -> 0
- net Net-(J11-Pad6): track 26.0 -> 0.00 mm
- net Net-(J11-Pad19): track 0.00 -> 22.8 mm
- net Net-(R4-Pad2): track 0.00 -> 22.5 mm
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
Commit message: Routing e Zone OK
Parts:
- added TP31: Pulse Generator, SerigrafieMakerLab:Disp4x7Seg, F.Cu at (186.9, 121.6)
- added TP32: Pulse Generator, SerigrafieMakerLab:Disp4x7Seg, F.Cu at (228.2, 81.3)
- added TP34: Pulse Generator, SerigrafieMakerLab:Disp4x7Seg, F.Cu at (228.2, 11.8)
- added TP35: Pulse Generator, SerigrafieMakerLab:Disp4x7Seg, F.Cu at (228.2, 121.6)
- J11: value Conn_02x10_Counter_Clockwise -> 1 2 3 4 5
- moved J24 1.88 mm to (221.8, 120.1)
- moved J23 1.88 mm to (248.4, 120.1)
- moved J22 1.88 mm to (258.2, 120.2)
- moved TP26 0.11 mm to (80.7, 30.1)
Routing:
- net GND: vias 128 -> 146

Commit message: Up Serigrafie
Parts:
- J11: value 1 2 3 4 5 -> Gnd Dp a b c d e f g
- J9: value Conn_02x05_Counter_Clockwise -> D C B A LE
