File: Kc/MakerLAB_r03C/Gen_Clock.kicad_sch (KiCad schematic)
At the start: 15 parts, among them J17 Conn_02x10_Counter_Clockwise, J26 Conn_01x06_Female, SW5 SW_Rotary12, U7 NE555P

Commit message: 20230404 14:30
Parts:
- removed J17: Conn_02x10_Counter_Clockwise, Connector_PinHeader_2.54mm:PinHeader_2x10_P2.54mm_Vertical, symbol Connector_Generic:Conn_02x10_Counter_Clockwise
- added J3: Conn_02x10_Counter_Clockwise, Connector_PinSocket_2.54mm:PinSocket_2x10_P2.54mm_Vertical, symbol Connector_Generic:Conn_02x10_Odd_Even
Connections:
- net +5V: now also J3.15 (Pin_15), J3.16 (Pin_16), J3.17 (Pin_17), J3.18 (Pin_18), J3.19 (Pin_19), J3.20 (Pin_20)
- net GND: now also J3.1 (Pin_1), J3.2 (Pin_2), J3.3 (Pin_3), J3.4 (Pin_4), J3.5 (Pin_5), J3.6 (Pin_6)
- net at D17.1 (K), U7.3 (Q): now also J3.10 (Pin_10), J3.11 (Pin_11), J3.12 (Pin_12), J3.13 (Pin_13), J3.14 (Pin_14), J3.7 (Pin_7), J3.8 (Pin_8), J3.9 (Pin_9)

Commit message: SCHEMI CONN ANNOTATI
CONNETTORI ANNOTATI 5.4.23
Parts:
- J3: value Conn_02x10_Counter_Clockwise -> GND CLOCK +5V
Changed lines of the file:
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@@
     (in_bom yes) (on_board yes) (fields_autoplaced)
     (property "Reference" "J3" (id 0) (at 177.8 33.02 0))
-    (property "Value" "Conn_02x10_Counter_Clockwise" (id 1) (at 177.8 35.56 0))
+    (property "Value" "GND   CLOCK     +5V" (id 1) (at 177.8 35.56 0))
     (property "Footprint" "Connector_PinSocket_2.54mm:PinSocket_2x10_P2.54mm_Vertical" (id 2) (at 179.07 49.53 0)
       (effects (font (size 1.27 1.27)) hide)
