File: Kc/MakerLAB_r03C/Gen_Fronti_sch.kicad_sch (KiCad schematic)
At the start: 10 parts, among them J2 Conn_02x05_Counter_Clockwise, SW6 SW_Push, SW7 SW_Push, U8 74LS00

Commit message: SCHEMI CONN ANNOTATI
CONNETTORI ANNOTATI 5.4.23
Parts:
- J2: value Conn_02x05_Counter_Clockwise -> Gnd FP6 FP7
Changed lines of the file:
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@@
     (in_bom yes) (on_board yes)
     (property "Reference" "J2" (id 0) (at 175.26 50.8 0))
-    (property "Value" "Conn_02x05_Counter_Clockwise" (id 1) (at 176.53 53.34 0))
+    (property "Value" "Gnd  FP6  FP7" (id 1) (at 176.53 53.34 0))
     (property "Footprint" "Connector_PinSocket_2.54mm:PinSocket_2x05_P2.54mm_Vertical" (id 2) (at 173.99 64.77 0)
       (effects (font (size 1.27 1.27)) hide)
