File: Kc/MakerLAB_r03C/MakerLAB_r03C.kicad_sch (KiCad schematic)
At the start: 4 parts

Commit message: r03C
Parts:
- +5, +Var1, GND1: footprint (none) -> Connector_PinHeader_2.54mm:PinHeader_1x05_P2.54mm_Vertical
Changed lines of the file:
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@@
     (property "Reference" "+5" (id 0) (at 24.13 46.99 0))
     (property "Value" "Conn_01x05" (id 1) (at 24.13 45.72 0))
-    (property "Footprint" "" (id 2) (at 24.13 54.61 0)
+    (property "Footprint" "Connector_PinHeader_2.54mm:PinHeader_1x05_P2.54mm_Vertical" (id 2) (at 24.13 54.61 0)
       (effects (font (size 1.27 1.27)) hide)
     )
@@
     (property "Reference" "+Var1" (id 0) (at 24.13 86.36 0))
     (property "Value" "Conn_01x05" (id 1) (at 24.13 85.09 0))
-    (property "Footprint" "" (id 2) (at 24.13 93.98 0)
+    (property "Footprint" "Connector_PinHeader_2.54mm:PinHeader_1x05_P2.54mm_Vertical" (id 2) (at 24.13 93.98 0)
       (effects (font (size 1.27 1.27)) hide)
     )
@@
     (property "Reference" "GND1" (id 0) (at 24.13 123.19 0))
     (property "Value" "Conn_01x05" (id 1) (at 24.13 121.92 0))
-    (property "Footprint" "" (id 2) (at 24.13 130.81 0)
+    (property "Footprint" "Connector_PinHeader_2.54mm:PinHeader_1x05_P2.54mm_Vertical" (id 2) (at 24.13 130.81 0)
       (effects (font (size 1.27 1.27)) hide)
     )
@@
       (reference "#PWR044") (unit 1) (value "GND") (footprint "")
     )
-    (path "/1c7b6ba1-9bc1-4836-88a5-b185a760b165/0069c09e-d3cd-44b5-a43b-a9515ffdba45"
-      (reference "#PWR0101") (unit 1) (value "GNDA") (footprint "")
+    (path "/1c7b6ba1-9bc1-4836-88a5-b185a760b165/f619d527-b4ab-444b-9874-6e2ffe5f2b60"
+      (reference "#PWR0101") (unit 1) (value "GND") (footprint "")
     )
     (path "/3c0235f3-a875-43f2-8c96-ee177e52f2ff"
@@
     )
     (path "/248009d1-f2be-4cb2-83d3-96998f7e00ec"
-      (reference "+5") (unit 1) (value "Conn_01x05") (footprint "")
+      (reference "+5") (unit 1) (value "Conn_01x05") (footprint "Connector_PinHeader_2.54mm:PinHeader_1x05_P2.54mm_Vertical")
     )
     (path "/71e26261-99a6-40c7-adb8-51200aca824b"
-      (reference "+Var1") (unit 1) (value "Conn_01x05") (footprint "")
+      (reference "+Var1") (unit 1) (value "Conn_01x05") (footprint "Connector_PinHeader_2.54mm:PinHeader_1x05_P2.54mm_Vertical")
     )
     (path "/7b083e6b-8037-4945-a6a7-d033f55692d8/c3dc9d45-d241-4d18-a10c-751ce53835ca"
@@
     )
     (path "/62ab733d-ee67-4f7c-8a1e-1b8f9ec01131/42e66396-2231-4ff9-b7ba-e74ad7c44ef5"
-      (reference "C13") (unit 1) (value "100nF") (footprint "")
-    )
-    (path "/62ab733d-ee67-4f7c-8a1e-1b8f9ec01131/5c5d14d1-b0db-4760-a228-ee0599d58036"
-      (reference "C14") (unit 1) (value "C_Polarized") (footprint "")
+      (reference "C13") (unit 1) (value "100nF") (footprint "Capacitor_THT:C_Axial_L5.1mm_D3.1mm_P7.50mm_Horizontal")
     )
     (path "/62ab733d-ee67-4f7c-8a1e-1b8f9ec01131/b8e78b2c-6934-41f1-910d-a4ea6ebf6af9"
-      (reference "C15") (unit 1) (value "10nF") (footprint "")
+      (reference "C15") (unit 1) (value "10nF") (footprint "Capacitor_THT:C_Axial_L5.1mm_D3.1mm_P7.50mm_Horizontal")
     )
     (path "/fab53e88-89c0-40b1-9c44-f0dadc28ccb9/5059abb7-0788-45bb-9110-9015d0b71e00"
@@
     )
     (path "/9c3b1e88-f55e-4bc3-b91f-af287aafcdc0"
-      (reference "GND1") (unit 1) (value "Conn_01x05") (footprint "")
+      (reference "GND1") (unit 1) (value "Conn_01x05") (footprint "Connector_PinHeader_2.54mm:PinHeader_1x05_P2.54mm_Vertical")
     )
     (path "/fab53e88-89c0-40b1-9c44-f0dadc28ccb9/14ffdc75-9d3c-49c1-ac7d-d9151c9aad0b"
@@
     )
     (path "/3fdafdb4-8fb2-4faf-beb8-83b0478cdff5/c7807945-7702-4701-ae9a-fdd3c32f0f94"
-      (reference "R4") (unit 1) (value "330") (footprint "")
+      (reference "R4") (unit 1) (value "330") (footprint "Resistor_THT:R_Axial_DIN0207_L6.3mm_D2.5mm_P10.16mm_Horizontal")
     )
     (path "/3fdafdb4-8fb2-4faf-beb8-83b0478cdff5/df3c641e-4ee8-4a98-b360-520bb86cd1da"
@@
     )
     (path "/1c7b6ba1-9bc1-4836-88a5-b185a760b165/fff0659a-c646-48a3-89d6-f5f650ef59bc"
-      (reference "TP29") (unit 1) (value "8 x LED") (footprint "SerigrafieMakerLAB:Clock NE555")
+      (reference "TP29") (unit 1) (value "8 x LED") (footprint "SerigrafieMakerLab:Clock NE555")
     )
     (path "/1c7b6ba1-9bc1-4836-88a5-b185a760b165/df6c0773-6376-4e47-b98b-9de65ed6dc0a"
