File: Kc/MakerLAB_r03C/OLED_128x64.kicad_sch (KiCad schematic)
At the start: 4 parts, among them J21 Conn_01x03

Commit message: SCHEMI CONN ANNOTATI
CONNETTORI ANNOTATI 5.4.23
Parts:
- J21: value Conn_01x03 -> Gnd SCL SDA
Changed lines of the file:
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@@
       (effects (font (size 1.27 1.27)) (justify right))
     )
-    (property "Value" "Conn_01x03" (id 1) (at 142.24 53.3399 90)
+    (property "Value" "Gnd SCL SDA" (id 1) (at 142.24 53.3399 90)
       (effects (font (size 1.27 1.27)) (justify right))
     )
