File: Kc/MakerLAB_r03C/Pulse_2.kicad_sch (KiCad schematic)
At the start: 14 parts, among them J16 Conn_02x05_Counter_Clockwise, SW3 SW_Push, SW4 SW_Push, U6 74LS14

Commit message: SCHEMI CONN ANNOTATI
CONNETTORI ANNOTATI 5.4.23
Parts:
- J16: value Conn_02x05_Counter_Clockwise -> GND P3 P4
Changed lines of the file:
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@@
     (in_bom yes) (on_board yes)
     (property "Reference" "J16" (id 0) (at 185.42 48.26 0))
-    (property "Value" "Conn_02x05_Counter_Clockwise" (id 1) (at 186.69 50.8 0))
+    (property "Value" "GND  P3   P4" (id 1) (at 186.69 50.8 0))
     (property "Footprint" "Connector_PinSocket_2.54mm:PinSocket_2x05_P2.54mm_Vertical" (id 2) (at 184.15 62.23 0)
       (effects (font (size 1.27 1.27)) hide)
