File: Kc/MakerLAB_r03C/Visual2dgt.kicad_sch (KiCad schematic)
At the start: 12 parts, among them J19 Conn_01x10_Female, U10 9368, U9 9368

Commit message: SCHEMI CONN ANNOTATI
CONNETTORI ANNOTATI 5.4.23
Parts:
- J19: value Conn_01x10_Female -> LE A0 A1 A2 A3 A0 A1 A2 A3 LE
Changed lines of the file:
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@@
     (in_bom yes) (on_board yes)
     (property "Reference" "J19" (id 0) (at 40.64 63.5 90))
-    (property "Value" "Conn_01x10_Female" (id 1) (at 43.18 64.77 90))
+    (property "Value" "LE A0 A1 A2 A3 A0 A1 A2 A3 LE" (id 1) (at 43.18 64.77 90))
     (property "Footprint" "Connector_PinHeader_2.54mm:PinHeader_1x10_P2.54mm_Vertical" (id 2) (at 45.72 66.04 0)
       (effects (font (size 1.27 1.27)) hide)
