File: Kc/MakerLAB_r03D/Visual_8Led.kicad_sch (KiCad schematic)
At the start: 21 parts, among them J13 GND 0 1 2 3 4 5 6 7 +5V, J14 8Bit Jumper, U5 ULN2803A

Commit message: Versione D prima del controllo di fine sessione
Parts:
- RN1: value Resistor Array -> 330
Changed lines of the file:
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@@
     (in_bom yes) (on_board yes) (fields_autoplaced)
     (property "Reference" "RN1" (id 0) (at 156.21 81.28 90))
-    (property "Value" "Resistor Array" (id 1) (at 156.21 83.82 90))
+    (property "Value" "330" (id 1) (at 156.21 83.82 90))
     (property "Footprint" "Package_DIP:DIP-16_W7.62mm_Socket_LongPads" (id 2) (at 156.21 109.855 90)
       (effects (font (size 1.27 1.27)) hide)
