File: Kc/MakerLAB_r03D/MakerLAB_r03D.kicad_pcb (KiCad board)
At the start: 2 copper layers, 374 x 178 mm, 183 parts, among them J1 Fix-Mod, J11 Gnd Dp a b c d e f g, J12 Conn_02x05_Counter_Clockwise, J13 GND 0 1 2 3 4 5 6 7 +5V, J14 8Bit Jumper, J15 GND 0 1 2 3 4 5 6 7 +5V, J16 Conn_02x05_Counter_Clockwise, J19 LE A0 A1 A2 A3 A0 A1 A2 A3 LE, J2 Conn_02x05_Counter_Clockwise, J21 Conn_01x03, J22 Conn_02x20_Counter_Clockwise, J23 Conn_02x20_Counter_Clockwise, J24 Conn_02x20_Counter_Clockwise, J25 IR Emitter & Sensor, J26 Conn_01x06_Female, J29 Conn_01x02_Male, J3 Conn_02x10_Counter_Clockwise, J30 Conn_01x02_Male, J33 Visible Light Sensor, J34 Conn_01x05, J4 Barrel_Jack_MountingPin, J5 Conn_01x02_Male, J9 A B C D LE, Q1 2N3904, Q2 2N3904, Q3 2N3904, Q4 2N3904, Q5 BC237, Q6 H21A1, Q7 BS170, Q8 BS170, SW1 SwGenerale, SW2 SW_DIP_x08, SW3 Down, SW4 Up, SW5 SW_Rotary12, SW6 Down, SW7 Up, U1 LM317_TO-220, U10 9368, U11 L78L33, U12 HC-05 (ZC142200), U2 LM7805_TO220, U3 DM9368, U4 CC56-12EWA, U5 ULN2803A, U6 74LS14, U7 NE555P, U8 74LS00, U9 9368

Commit message: Add files via upload
Parts:
- J11: value Gnd Dp a b c d e f g -> Gnd a b c d e f g
- J16: value Conn_02x05_Counter_Clockwise -> GND P3 P4
- J2: value Conn_02x05_Counter_Clockwise -> Gnd FP6 FP7
- J21: value Conn_01x03 -> Gnd SCL SDA
- J3: value Conn_02x10_Counter_Clockwise -> GND CLOCK +5V
- J9: value A B C D LE -> A B C D LE
- SW3, SW6: value Down -> SW_Push
- SW4, SW7: value Up -> SW_Push
- TP21: value Alimentatore Variabile -> Alimentaore Variabile
- TP29: value Gen.Clock -> 8 x LED
- TP34: value 2 * 7 Seg. -> Pulse Generator
- U11: value L78L33 -> L78L33_SOT89
Other:
- board text added: "B C D"
- board text added: "CC1 CC2"
- board text added: "CC3 CC4 GND"
- board text added: "Dpx"
- board text added: "GND Ex. Cap"
- board text added: "GND Rx Tx En State"
- board text added: "GND cc1 cc2"
- board text added: "LE A"
- board text added: "cc3 cc4"
Changed lines of the file:
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@@
     (descr "Through hole straight pin header, 1x05, 2.54mm pitch, single row")
     (tags "Through hole pin header THT 1x05 2.54mm single row")
-    (property "Sheetfile" "MakerLAB_r03C.kicad_sch")
+    (property "Sheetfile" "MakerLAB_r03D.kicad_sch")
     (property "Sheetname" "")
     (attr through_hole)
@@
     (descr "Through hole straight pin header, 1x05, 2.54mm pitch, single row")
     (tags "Through hole pin header THT 1x05 2.54mm single row")
-    (property "Sheetfile" "MakerLAB_r03C.kicad_sch")
+    (property "Sheetfile" "MakerLAB_r03D.kicad_sch")
     (property "Sheetname" "")
     (attr through_hole)
@@
       (effects (font (size 1 1) (thickness 0.15)))
     )
-    (fp_text value "Conn_02x05_Counter_Clockwise" (at 2.54 5.08 90) (layer "F.Fab")
+    (fp_text value "Gnd  FP6  FP7" (at 2.54 5.08 90) (layer "F.Fab")
       (effects (font (size 1 1) (thickness 0.15)))
     )
@@
       (effects (font (size 1 1) (thickness 0.15)))
     )
-    (fp_text value "Conn_01x03" (at 0 7.41) (layer "F.Fab")
+    (fp_text value "Gnd SCL SDA" (at -3.1496 2.6266 90) (layer "F.Fab")
       (effects (font (size 1 1) (thickness 0.15)))
     )
@@
       (effects (font (size 1 1) (thickness 0.15)))
     )
-    (fp_text value "Down" (at -5.3848 3.429) (layer "F.SilkS")
+    (fp_text value "SW_Push" (at -5.3848 3.429) (layer "F.SilkS")
       (effects (font (size 1.5 1.5) (thickness 0.375)))
     )
@@
       (effects (font (size 1 1) (thickness 0.15)))
     )
-    (fp_text value "2 * 7 Seg." (at 6.985 4.7498 unlocked) (layer "F.SilkS")
+    (fp_text value "Pulse Generator" (at 6.985 4.7498 unlocked) (layer "F.SilkS")
       (effects (font (size 1.5 1.5) (thickness 0.375)))
     )
@@
       (effects (font (size 1 1) (thickness 0.15)))
     )
-    (fp_text value "A B C D LE" (at 3.3582 3.78 90) (layer "F.SilkS")
+    (fp_text value "A  B  C  D  LE" (at 2.9264 5.2024 90) (layer "F.SilkS") hide
       (effects (font (size 1 1) (thickness 0.15)))
     )
@@
       (effects (font (size 1 1) (thickness 0.15)))
     )
-    (fp_text value "Conn_02x10_Counter_Clockwise" (at 2.667 10.8204 90) (layer "F.SilkS")
+    (fp_text value "GND    CLOCK      +5V" (at -5.588 10.8204 90) (layer "F.SilkS")
       (effects (font (size 1 1) (thickness 0.15)))
     )
@@
       (effects (font (size 1 1) (thickness 0.15)))
     )
-    (fp_text value "L78L33" (at -2.921 -6.9088 180) (layer "F.SilkS")
+    (fp_text value "L78L33_SOT89" (at -2.921 -6.9088 180) (layer "F.SilkS")
       (effects (font (size 1 1) (thickness 0.15)))
     )
@@
     (descr "Through hole straight pin header, 1x05, 2.54mm pitch, single row")
     (tags "Through hole pin header THT 1x05 2.54mm single row")
-    (property "Sheetfile" "MakerLAB_r03C.kicad_sch")
+    (property "Sheetfile" "MakerLAB_r03D.kicad_sch")
     (property "Sheetname" "")
     (attr through_hole)
@@
       (effects (font (size 1 1) (thickness 0.15)))
     )
-    (fp_text value "Conn_02x05_Counter_Clockwise" (at 2.833 6.4058 90) (layer "F.Fab")
+    (fp_text value "GND  P3   P4" (at 2.833 6.4058 90) (layer "F.Fab")
       (effects (font (size 1 1) (thickness 0.15)))
     )
@@
       (effects (font (size 1 1) (thickness 0.15)))
     )
-    (fp_text value "Alimentatore Variabile" (at 19.812 -3.9624 unlocked) (layer "F.SilkS")
+    (fp_text value "Alimentaore Variabile" (at 19.812 -3.9624 unlocked) (layer "F.SilkS")
       (effects (font (size 1.5 1.5) (thickness 0.375)))
     )
@@
       (effects (font (size 1 1) (thickness 0.15)))
     )
-    (fp_text value "Up" (at -4.4332 1.6714 180) (layer "F.SilkS")
+    (fp_text value "SW_Push" (at -4.4332 1.6714 180) (layer "F.SilkS")
       (effects (font (size 1.5 1.5) (thickness 0.375)))
     )
@@
       (effects (font (size 1 1) (thickness 0.15)))
     )
-    (fp_text value "Gnd Dp a  b  c  d   e   f   g  " (at 2.9772 13.7114 180) (layer "F.SilkS")
-      (effects (font (size 1 1) (thickness 0.15)))
+    (fp_text value "Gnd      a  b  c  d   e   f   g  " (at -5.0746 12.797 180) (layer "F.SilkS")
+      (effects (font (size 1 1) (thickness 0.2)))
     )
     (fp_text user "${REFERENCE}" (at -1.27 11.43) (layer "F.SilkS")
@@
       (effects (font (size 1 1) (thickness 0.15)))
     )
-    (fp_text value "Conn_02x05_Counter_Clockwise" (at 2.6216 4.6944 180) (layer "F.SilkS")
+    (fp_text value "Conn_02x05_Counter_Clockwise" (at 2.6216 4.6944 180) (layer "F.SilkS") hide
       (effects (font (size 1 1) (thickness 0.15)))
     )
@@
       (effects (font (size 1 1) (thickness 0.15)))
     )
-    (fp_text value "Conn_01x05" (at -2.6924 4.44 90) (layer "F.Fab")
+    (fp_text value "Conn_01x05" (at -1.2192 3.7796 90) (layer "F.Fab") hide
       (effects (font (size 1 1) (thickness 0.15)))
     )
@@
       (effects (font (size 1 1) (thickness 0.15)))
     )
-    (fp_text value "Down" (at 15.0994 1.6206 180) (layer "F.SilkS")
+    (fp_text value "SW_Push" (at 15.0994 1.6206 180) (layer "F.SilkS")
       (effects (font (size 1.5 1.5) (thickness 0.375)))
     )
@@
       (effects (font (size 1 1) (thickness 0.15)))
     )
-    (fp_text value "Up" (at 11.0744 3.3274) (layer "F.SilkS")
+    (fp_text value "SW_Push" (at 11.0744 3.3274) (layer "F.SilkS")
       (effects (font (size 1.5 1.5) (thickness 0.375)))
     )
@@
     (descr "Through hole straight pin header, 1x05, 2.54mm pitch, single row")
     (tags "Through hole pin header THT 1x05 2.54mm single row")
-    (property "Sheetfile" "MakerLAB_r03C.kicad_sch")
+    (property "Sheetfile" "MakerLAB_r03D.kicad_sch")
     (property "Sheetname" "")
     (attr through_hole)
@@
       (effects (font (size 1 1) (thickness 0.15)))
     )
-    (fp_text value "Gen.Clock" (at 44.9586 17.8562 unlocked) (layer "F.SilkS")
+    (fp_text value "8 x LED" (at 44.9586 17.8562 unlocked) (layer "F.SilkS")
       (effects (font (size 1.5 1.5) (thickness 0.375)))
     )
@@
   (gr_circle (center 62.6872 159.3088) (end 76.494641 159.3088) (layer "F.SilkS") (width 0.1) (fill none))
   (gr_rect (start 0 0) (end 374 178) (layer "Edge.Cuts") (width 0.1) (fill none))
+  (gr_text "B\n\nC\n\nD" (at 179.578 39.37) (layer "F.SilkS")
+    (effects (font (size 1 1) (thickness 0.2)))
+  )
+  (gr_text "GND Rx Tx En State" (at 214.249 91.948 90) (layer "F.SilkS")
+    (effects (font (size 1 1) (thickness 0.2)))
+  )
+  (gr_text "LE\n\nA" (at 179.578 32.385) (layer "F.SilkS")
+    (effects (font (size 1 1) (thickness 0.2)))
+  )
+  (gr_text "GND cc1 cc2" (at 126.365 28.956) (layer "F.SilkS")
+    (effects (font (size 1 1) (thickness 0.2)))
+  )
+  (gr_text "GND     Ex. Cap" (at 179.705 153.162 90) (layer "F.SilkS")
+    (effects (font (size 1.2 1.2) (thickness 0.2)))
+  )
+  (gr_text "CC1\n \nCC2\n " (at 170.307 33.528) (layer "F.SilkS")
+    (effects (font (size 1 1) (thickness 0.2)))
+  )
+  (gr_text "CC3\n \nCC4\n \nGND" (at 170.18 39.497) (layer "F.SilkS")
+    (effects (font (size 1 1) (thickness 0.2)))
+  )
+  (gr_text "Dpx" (at 147.955 28.448) (layer "F.SilkS")
+    (effects (font (size 1 1) (thickness 0.2)))
+  )
+  (gr_text "cc3 cc4" (at 134.493 28.956) (layer "F.SilkS")
+    (effects (font (size 1 1) (thickness 0.2)))
+  )
   (segment (start 210.439 28.954) (end 208.234 31.159) (width 0.25) (layer "F.Cu") (net 1))
   (segment (start 209.042 20.955) (end 210.428 22.341) (width 0.25) (layer "F.Cu") (net 1))

Commit message: Versione D prima del controllo di fine sessione
Parts:
- J1: value Fix-Mod -> Fix
- J11: value Gnd a b c d e f g -> Gnd a b c d e f g
- J12: value Conn_02x05_Counter_Clockwise -> GND cc1 cc2
- J13: value GND 0 1 2 3 4 5 6 7 +5V -> GND 7 6 5 4 3 2 1 0 +5V
- J14: value 8Bit Jumper -> +5V 7 6 5 4 3 2 1 0 GND
- J15: value GND 0 1 2 3 4 5 6 7 +5V -> +5V 7 6 5 4 3 2 1 0 GND
- J19: value LE A0 A1 A2 A3 A0 A1 A2 A3 LE -> LeU A0 A1 A2 A3 A0 A1 A2 A3 LeD
- J23: value Conn_02x20_Counter_Clockwise -> 1
- RN1: value Resistor Array -> 330
- SW3, SW6: value SW_Push -> Down
- SW4, SW7: value SW_Push -> Up
- TP29: value 8 x LED -> Clock Gen.
- TP34: value Pulse Generator -> 2*7 Segmenti
- Uni-A4: value Jumper_3_Open -> Zero Decine
- moved C22 7.00 mm to (238.9, 26.1), turned to 180 degrees
Connections:
- J33 pad 1: Net-(J33-Pad1) -> GND
- R29 pad 2: Net-(J33-Pad1) -> GND
- R31 pad 2: Net-(J33-Pad1) -> GND
Routing:
- net Net-(J33-Pad1): track 25.8 -> 0.00 mm
- net Net-(J15-Pad5): track 47.3 -> 50.7 mm
- net Net-(J15-Pad4): track 44.4 -> 47.4 mm
- net /Alimentazione/+5V: track 1521.8 -> 1524.8 mm
- net Net-(J15-Pad6): track 48.6 -> 51.0 mm
- net Net-(J15-Pad3): track 41.2 -> 43.4 mm
- net Net-(J15-Pad7): track 45.3 -> 47.1 mm
- net Net-(J15-Pad8): track 42.0 -> 43.0 mm
- net Net-(J14-Pad19): track 26.4 -> 27.4 mm
Other:
- board text removed: "B C D"
- board text removed: "CC1 CC2"
- board text removed: "CC3 CC4 GND"
- board text removed: "Dpx"
- board text removed: "GND Ex. Cap"
- board text removed: "GND cc1 cc2"
- board text removed: "LE A"
- board text removed: "cc3 cc4"

Commit message: Fine Controllo
Parts:
- J3: value GND CLOCK +5V -> GND CLOCK +5V
Changed lines of the file:
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@@
       (effects (font (size 1 1) (thickness 0.15)))
     )
+    (fp_text user "|" (at 0.0459 -2.4588 180 unlocked) (layer "F.SilkS")
+      (effects (font (size 6 1) (thickness 0.3)))
+    )
     (fp_text user "${REFERENCE}" (at 0 5.08 90) (layer "F.Fab")
       (effects (font (size 1 1) (thickness 0.15)))
@@
       (effects (font (size 1 1) (thickness 0.15)))
     )
+    (fp_text user "|" (at 0 -2.3876 180 unlocked) (layer "F.SilkS")
+      (effects (font (size 6 1) (thickness 0.3)))
+    )
     (fp_text user "${REFERENCE}" (at 0 5.08 90) (layer "F.Fab")
       (effects (font (size 1 1) (thickness 0.15)))
@@
       (effects (font (size 1 1) (thickness 0.15)))
     )
-    (fp_text value "GND    CLOCK      +5V" (at -5.588 10.8204 90) (layer "F.SilkS")
-      (effects (font (size 1 1) (thickness 0.15)))
+    (fp_text value "GND      CLOCK      +5V" (at -6.1214 10.8712 90) (layer "F.SilkS")
+      (effects (font (size 1 1) (thickness 0.2)))
+    )
+    (fp_text user "]" (at -4.9784 11.8618 unlocked) (layer "F.SilkS")
+      (effects (font (size 4.5 1) (thickness 0.2)))
     )
-    (fp_text user "${REFERENCE}" (at -1.27 11.43 90) (layer "F.Fab")
+    (fp_text user "]" (at -4.9784 20.6248 unlocked) (layer "F.SilkS")
+      (effects (font (size 3.5 1) (thickness 0.2)))
+    )
+    (fp_text user "]" (at -4.9784 3.302 unlocked) (layer "F.SilkS")
+      (effects (font (size 3.5 1) (thickness 0.2)))
+    )
+    (fp_text user "${REFERENCE}" (at -1.27 11.43 90) (layer "F.Fab") hide
       (effects (font (size 1 1) (thickness 0.15)))
     )
@@
       (effects (font (size 1 1) (thickness 0.15)))
     )
+    (fp_text user "|" (at 0 -1.778 180 unlocked) (layer "F.SilkS")
+      (effects (font (size 3 1) (thickness 0.3)))
+    )
     (fp_text user "${REFERENCE}" (at 0 5.08 90) (layer "F.Fab")
       (effects (font (size 1 1) (thickness 0.15)))
@@
       (effects (font (size 1 1) (thickness 0.15)))
     )
+    (fp_text user "|" (at 0.0303 -1.7272 180 unlocked) (layer "F.SilkS")
+      (effects (font (size 3 1) (thickness 0.3)))
+    )
     (fp_text user "${REFERENCE}" (at 0 5.08 90) (layer "F.Fab")

Commit message: Ultima prima del logo
Parts:
- J16: value GND P3 P4 -> P3 P4
- J2: value Gnd FP6 FP7 -> FP6 FP7
- moved TP34 0.07 mm to (228.1, 11.8)
Changed lines of the file:
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@@
       (effects (font (size 1 1) (thickness 0.15)))
     )
-    (fp_text value "LED" (at 1.27 2.96 90) (layer "F.Fab")
+    (fp_text value "LED" (at -0.1778 2.921 90) (layer "F.Fab")
       (effects (font (size 1 1) (thickness 0.15)))
     )
@@
     (property "Sheetname" "Pulse_2")
     (attr through_hole)
-    (fp_text reference "C11" (at 5.456 -2.4756 90) (layer "F.SilkS")
+    (fp_text reference "C11" (at 2.2302 -2.3232 90) (layer "F.SilkS")
       (effects (font (size 1 1) (thickness 0.15)))
     )
-    (fp_text value "1uF" (at 1.7222 -2.3994 90) (layer "F.SilkS")
+    (fp_text value "1uF" (at -0.9956 -2.2216 90) (layer "F.SilkS")
       (effects (font (size 1 1) (thickness 0.15)))
     )
@@
       (effects (font (size 1 1) (thickness 0.15)))
     )
-    (fp_text value "Gnd  FP6  FP7" (at 2.54 5.08 90) (layer "F.Fab")
-      (effects (font (size 1 1) (thickness 0.15)))
+    (fp_text value "FP6   FP7" (at 3.1296 6.2184 90) (layer "F.SilkS")
+      (effects (font (size 1 1) (thickness 0.2)))
+    )
+    (fp_text user "]" (at 2.2406 8.7838 180 unlocked) (layer "F.SilkS")
+      (effects (font (size 1.75 1) (thickness 0.2)))
+    )
+    (fp_text user "]" (at 2.139 3.6784 180 unlocked) (layer "F.SilkS")
+      (effects (font (size 1.75 1) (thickness 0.2)))
+    )
+    (fp_text user "GND" (at 2.5962 -0.0046 90 unlocked) (layer "F.SilkS")
+      (effects (font (size 1 1) (thickness 0.2)))
     )
     (fp_text user "${REFERENCE}" (at -1.27 5.08 90) (layer "F.Fab")
@@
       (effects (font (size 1 1) (thickness 0.15)))
     )
-    (fp_text value "Gnd SCL SDA" (at -3.1496 2.6266 90) (layer "F.Fab")
+    (fp_text value "Gnd SCL SDA" (at -3.1496 2.6266 90) (layer "F.SilkS")
       (effects (font (size 1 1) (thickness 0.15)))
     )
@@
   )
   (footprint "SerigrafieMakerLab:Disp4x7Seg" (layer "F.Cu")
-    (at 228.1682 11.8364)
+    (at 228.116 11.7856)
     (property "Sheetfile" "PadSerigrafie.kicad_sch")
     (property "Sheetname" "Pad e Serigrafie")
@@
     (property "Sheetname" "Visual2dgt")
     (attr through_hole)
-    (fp_text reference "U10" (at 10.4072 1.4938 180) (layer "F.SilkS")
+    (fp_text reference "U10" (at 10.4326 12.6698 180) (layer "F.SilkS")
       (effects (font (size 1 1) (thickness 0.15)))
     )
-    (fp_text value "9368" (at 10.458 6.6246 180) (layer "F.SilkS")
+    (fp_text value "9368" (at 10.4834 17.8006 180) (layer "F.SilkS")
       (effects (font (size 1 1) (thickness 0.15)))
     )
@@
       (effects (font (size 1 1) (thickness 0.15)))
     )
-    (fp_text value "IR Emitter & Sensor" (at 17.0942 5.334) (layer "F.SilkS")
+    (fp_text value "IR Emitter & Sensor" (at 17.6022 5.3848) (layer "F.SilkS")
       (effects (font (size 1.5 1.5) (thickness 0.375)))
     )
@@
       (effects (font (size 1 1) (thickness 0.15)))
     )
+    (fp_text user "Un." (at -3.7034 5.0398 unlocked) (layer "F.SilkS")
+      (effects (font (size 1.5 1.5) (thickness 0.375)))
+    )
     (fp_text user "${REFERENCE}" (at 7.87 5.08 90) (layer "F.SilkS")
       (effects (font (size 1 1) (thickness 0.15)))
@@
       (effects (font (size 1 1) (thickness 0.15)))
     )
-    (fp_text value "GND  P3   P4" (at 2.833 6.4058 90) (layer "F.Fab")
-      (effects (font (size 1 1) (thickness 0.15)))
+    (fp_text value "P3    P4" (at 2.9092 5.9486 90) (layer "F.SilkS")
+      (effects (font (size 1 1) (thickness 0.2)))
+    )
+    (fp_text user "]" (at 2.1218 8.7426 180 unlocked) (layer "F.SilkS")
+      (effects (font (size 1.75 1) (thickness 0.2)))
+    )
+    (fp_text user "]" (at 2.071 3.7134 180 unlocked) (layer "F.SilkS")
+      (effects (font (size 1.75 1) (thickness 0.2)))
+    )
+    (fp_text user "GND" (at 2.7568 0.1066 90 unlocked) (layer "F.SilkS")
+      (effects (font (size 1 1) (thickness 0.2)))
     )
     (fp_text user "${REFERENCE}" (at -1.27 5.08 90) (layer "F.Fab")
@@
       (effects (font (size 2.5 2.5) (thickness 0.45)))
     )
-    (fp_text user "Hardware r03C" (at 14.605 -0.635 unlocked) (layer "F.SilkS")
+    (fp_text user "Hardware r03D" (at 14.605 -0.635 unlocked) (layer "F.SilkS")
       (effects (font (size 1 1) (thickness 0.15)))
     )
@@
       (effects (font (size 1 1) (thickness 0.15)))
     )
+    (fp_text user "Dec." (at -3.551 4.8212 unlocked) (layer "F.SilkS")
+      (effects (font (size 1.5 1.5) (thickness 0.375)))
+    )
     (fp_text user "${REFERENCE}" (at 7.87 5.08 90) (layer "F.SilkS")
